File: eagle-files/design1.brd (EAGLE design)
At the start: 60 x 20 mm, 77 parts, among them IC12 NRF52832, IC2 STM32L011F3U6TR, IC3 TPS54308DDCR, IC4 MCP6486T-E/OT, Q1 BSS138, Q2 SI3481DV, U1 MAX5422ETA-T, X1 DG3XX-02-5.0, Y1 32MHz, Y2 32.768kHz

Commit message: update pcb
Parts:
- removed U1: MAX5422ETA-T, MAX5422ETA-T:SON65P300X300X80-9N
- added D4: (no value), diode:SOD323-R
- added LS3: MIC94081YFT-TR, MIC94081YFT-TR:IC_MIC94081YFT-TR
- added R16: 47k, microbuilder:0603
Connections:
- net P18 renamed SWO/TDO
- net P26 renamed I2C_SDA
- net P27 renamed I2C_SCL
- removed net P15: IC12.18
- removed net P19: IC12.22
- new net WAKE-UP: D4.C, IC12.22, R16.2
- net 3.3V: no longer U1.1
- net GND: now also D4.A, LS3.2; no longer U1.5, U1.9
- net LED: now also IC12.18; no longer IC12.20
- net N$10: now also R16.1
- net PWM-CHG: now also IC12.20
- net VDD_BLE: now also LS3.3
Changed lines of the file:
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@@
 <?xml version="1.0" encoding="utf-8"?>
 <!DOCTYPE eagle SYSTEM "eagle.dtd">
-<eagle version="9.6.2">
+<eagle version="9.5.1">
 <drawing>
 <settings>
@@
 <attribute name="VALUE" x="-7.18185" y="-62.918975" size="0.4064" layer="27" ratio="10"/>
 </element>
-<element name="U1" library="MAX5422ETA-T" package="SON65P300X300X80-9N" value="MAX5422ETA-T" x="-5.756275" y="-67.052825" smashed="yes">
-<attribute name="AVAILABILITY" value="In Stock" x="-5.756275" y="-67.052825" size="1.778" layer="27" display="off"/>
-<attribute name="DESCRIPTION" value=" Digital Potentiometer 50k Ohm 1 Circuit 256 Taps SPI Interface 8-TDFN-EP (3x3) " x="-5.756275" y="-67.052825" size="1.778" layer="27" display="off"/>
-<attribute name="MF" value="Analog Devices" x="-5.756275" y="-67.052825" size="1.778" layer="27" display="off"/>
-<attribute name="MP" value="MAX5422ETA" x="-5.756275" y="-67.052825" size="1.778" layer="27" display="off"/>
-<attribute name="NAME" x="-8.066275" y="-65.325825" size="1.27" layer="25"/>
-<attribute name="PACKAGE" value="TDFN-EP-8 Maxim" x="-5.756275" y="-67.052825" size="1.778" layer="27" display="off"/>
-<attribute name="PRICE" value="None" x="-5.756275" y="-67.052825" size="1.778" layer="27" display="off"/>
-<attribute name="PURCHASE-URL" value="https://pricing.snapeda.com/search?q=MAX5422ETA&amp;ref=eda" x="-5.756275" y="-67.052825" size="1.778" layer="27" display="off"/>
-<attribute name="VALUE" x="-8.066275" y="-68.779825" size="1.27" layer="27" align="top-left"/>
-</element>
 <element name="C7" library="microbuilder" package="0603" value="10u" x="-6.8453" y="-71.5645" smashed="yes">
 <attribute name="NAME" x="-5.0673" y="-71.6915" size="0.8128" layer="25" font="vector" ratio="18"/>
@@
 <attribute name="NAME" x="-10.5791" y="-69.643625" size="0.6096" layer="25" font="vector" ratio="20" align="bottom-center"/>
 <attribute name="VALUE" x="-10.5791" y="-71.929625" size="0.6096" layer="27" font="vector" ratio="20" align="top-center"/>
+</element>
+<element name="D4" library="diode" library_urn="urn:adsk.eagle:library:210" package="SOD323-R" package3d_urn="urn:adsk.eagle:package:43437/1" value="" x="-15.401925" y="-75.765025" smashed="yes">
+<attribute name="NAME" x="-16.501925" y="-74.765025" size="1.27" layer="25"/>
+<attribute name="POPULARITY" value="4" x="-15.401925" y="-75.765025" size="1.778" layer="27" display="off"/>
+<attribute name="VALUE" x="-16.501925" y="-78.065025" size="1.27" layer="27"/>
+</element>
+<element name="R16" library="microbuilder" package="0603" value="47k" x="-15.401925" y="-77.943075" smashed="yes">
+<attribute name="NAME" x="-13.623925" y="-78.070075" size="0.8128" layer="25" font="vector" ratio="18"/>
+<attribute name="VALUE" x="-13.623925" y="-78.705075" size="0.4064" layer="27" font="vector" ratio="10"/>
+</element>
+<element name="LS3" library="MIC94081YFT-TR" package="IC_MIC94081YFT-TR" value="MIC94081YFT-TR" x="-15.24635" y="-81.21015" smashed="yes">
+<attribute name="AVAILABILITY" value="In Stock" x="-15.24635" y="-81.21015" size="1.778" layer="27" display="off"/>
+<attribute name="DESCRIPTION" value=" Power Switch/Driver 1:1 P-Channel 2A 4-TMLF® (0.85x0.85) " x="-15.24635" y="-81.21015" size="1.778" layer="27" display="off"/>
+<attribute name="MF" value="Microchip" x="-15.24635" y="-81.21015" size="1.778" layer="27" display="off"/>
+<attribute name="MP" value="MIC94081YFT-TR" x="-15.24635" y="-81.21015" size="1.778" layer="27" display="off"/>
+<attribute name="NAME" x="-16.49635" y="-80.21015" size="0.6096" layer="25"/>
+<attribute name="PACKAGE" value="UFDFN-4 Microchip" x="-15.24635" y="-81.21015" size="1.778" layer="27" display="off"/>
+<attribute name="PRICE" value="None" x="-15.24635" y="-81.21015" size="1.778" layer="27" display="off"/>
+<attribute name="VALUE" x="-16.49635" y="-82.21015" size="0.6096" layer="27" align="top-left"/>
 </element>
 </elements>
@@
 <contactref element="UPDATE" pad="1"/>
 <contactref element="C29" pad="2"/>
-<contactref element="U1" pad="5"/>
-<contactref element="U1" pad="9"/>
 <contactref element="C7" pad="2"/>
 <contactref element="JP5" pad="1"/>
+<contactref element="D4" pad="A"/>
+<contactref element="LS3" pad="2"/>
+<wire x1="-14.301925" y1="-75.765025" x2="-15.44635" y2="-81.41015" width="0" layer="19" extent="1-1"/>
+<wire x1="-11.3919" y1="-70.786625" x2="-14.301925" y2="-75.765025" width="0" layer="19" extent="1-1"/>
 <wire x1="-5.9953" y1="-71.5645" x2="-11.3919" y2="-70.786625" width="0" layer="19" extent="1-1"/>
-<wire x1="-4.271275" y1="-68.027825" x2="-5.9953" y2="-71.5645" width="0" layer="19" extent="1-1"/>
-<wire x1="-5.756275" y1="-67.052825" x2="-4.271275" y2="-68.027825" width="0" layer="19" extent="1-1"/>
-<wire x1="-1.627875" y1="-55.229125" x2="-5.756275" y2="-67.052825" width="0" layer="19" extent="1-1"/>
+<wire x1="-1.627875" y1="-55.229125" x2="-5.9953" y2="-71.5645" width="0" layer="19" extent="1-1"/>
 <wire x1="-1.0169" y1="-51.96205" x2="-1.627875" y2="-55.229125" width="0" layer="19" extent="1-1"/>
 <wire x1="-1.8246" y1="-49.317275" x2="-1.0169" y2="-51.96205" width="0" layer="19" extent="1-1"/>
@@
 <wire x1="12.912725" y1="2.644775" x2="12.915" y2="2.6425" width="0.254" layer="1"/>
 <wire x1="12.915" y1="2.6425" x2="13.97" y2="2.6425" width="0.254" layer="1"/>
-<contactref element="U1" pad="1"/>
-<wire x1="11.745" y1="2.4925" x2="-7.241275" y2="-66.077825" width="0" layer="19" extent="1-1"/>
 </signal>
 <signal name="SWDCLK">
@@
 <wire x1="50.71745" y1="6.378575" x2="55.591075" y2="6.378575" width="0.254" layer="1"/>
 <wire x1="55.591075" y1="6.378575" x2="56.8325" y2="7.62" width="0.254" layer="1"/>
-<contactref element="IC12" pad="20"/>
-<wire x1="-4.533975" y1="-25.05165" x2="49.815" y2="6.62" width="0" layer="19" extent="1-1"/>
+<contactref element="IC12" pad="18"/>
+<wire x1="-5.333975" y1="-25.05165" x2="49.815" y2="6.62" width="0" layer="19" extent="1-1"/>
 </signal>
 <signal name="USART2_TX">
@@
 <wire x1="8.8925" y1="12.6325" x2="8.861575" y2="12.601575" width="0.254" layer="1"/>
 <wire x1="8.861575" y1="12.601575" x2="8.40105" y2="12.601575" width="0.254" layer="1"/>
+<contactref element="R16" pad="1"/>
+<wire x1="21.624925" y1="4.822825" x2="-16.251925" y2="-77.943075" width="0" layer="19" extent="1-1"/>
 </signal>
 <signal name="N$1">
@@
 <contactref element="IC12" pad="27"/>
 </signal>
-<signal name="P18">
+<signal name="SWO/TDO">
 <contactref element="IC12" pad="21"/>
 <contactref element="DEBUG1" pad="6"/>
@@
 <contactref element="IC12" pad="23"/>
 </signal>
-<signal name="P19">
-<contactref element="IC12" pad="22"/>
-</signal>
 <signal name="N$50">
 <contactref element="C77" pad="2"/>
@@
 <wire x1="-2.933975" y1="-19.13165" x2="-4.242825" y2="-52.58435" width="0" layer="19" extent="1-1"/>
 </signal>
-<signal name="P27">
+<signal name="I2C_SCL">
 <contactref element="IC12" pad="39"/>
 </signal>
-<signal name="P26">
+<signal name="I2C_SDA">
 <contactref element="C76" pad="2"/>
 <contactref element="IC12" pad="38"/>
@@
 <contactref element="UART_INTERFACE" pad="4"/>
 <wire x1="4.12115" y1="-34.2265" x2="-8.093975" y2="-23.09165" width="0" layer="19" extent="1-1"/>
-</signal>
-<signal name="P15">
-<contactref element="IC12" pad="18"/>
 </signal>
 <signal name="P16">
@@
 <contactref element="R50" pad="2"/>
 <contactref element="R60" pad="1"/>
-<wire x1="4.43955" y1="-57.56275" x2="-7.73645" y2="-49.317275" width="0" layer="19" extent="1-1"/>
+<contactref element="LS3" pad="3"/>
+<wire x1="4.43955" y1="-57.56275" x2="-15.04635" y2="-81.41015" width="0" layer="19" extent="1-1"/>
 <wire x1="6.13955" y1="-55.229125" x2="4.43955" y2="-57.56275" width="0" layer="19" extent="1-1"/>
 <wire x1="14.0852" y1="-45.4279" x2="6.13955" y2="-55.229125" width="0" layer="19" extent="1-1"/>
 <wire x1="15.03045" y1="-41.6941" x2="14.0852" y2="-45.4279" width="0" layer="19" extent="1-1"/>
 <wire x1="20.733775" y1="-45.4279" x2="14.0852" y2="-45.4279" width="0" layer="19" extent="1-1"/>
+<wire x1="-7.73645" y1="-49.317275" x2="4.43955" y2="-57.56275" width="0" layer="19" extent="1-1"/>
 <wire x1="12.861925" y1="-21.48205" x2="15.03045" y2="-41.6941" width="0" layer="19" extent="1-1"/>
 <wire x1="-2.173975" y1="-19.89165" x2="12.861925" y2="-21.48205" width="0" layer="19" extent="1-1"/>
@@
 <signal name="PWM-CHG">
 <contactref element="JP5" pad="3"/>
+<contactref element="IC12" pad="20"/>
+<wire x1="-4.533975" y1="-25.05165" x2="-9.7663" y2="-70.786625" width="0" layer="19" extent="1-1"/>
+</signal>
+<signal name="WAKE-UP">
+<contactref element="D4" pad="C"/>
+<contactref element="R16" pad="2"/>
+<contactref element="IC12" pad="22"/>
+<wire x1="-14.551925" y1="-77.943075" x2="-16.501925" y2="-75.765025" width="0" layer="19" extent="1-1"/>
+<wire x1="-3.733975" y1="-25.05165" x2="-16.501925" y2="-75.765025" width="0" layer="19" extent="1-1"/>
 </signal>
 </signals>
@@
 </board>
 </drawing>
+<compatibility>
+<note version="8.2" severity="warning">
+Since Version 8.2, EAGLE supports online libraries. The ids
+of those online libraries will not be understood (or retained)
+with this version.
+</note>
+<note version="8.3" severity="warning">
+Since Version 8.3, EAGLE supports URNs for individual library
+assets (packages, symbols, and devices). The URNs of those assets
+will not be understood (or retained) with this version.
+</note>
+<note version="8.3" severity="warning">
+Since Version 8.3, EAGLE supports the association of 3D packages
+with devices in libraries, schematics, and board files. Those 3D
+packages will not be understood (or retained) with this version.
+</note>
+</compatibility>
 </eagle>
