File: eagle-files/design1.sch (EAGLE design)
At the start: 95 parts, among them IC12 NRF52832, IC2 STM32L011F3U6TR, IC3 TPS54308DDCR, IC4 MCP6486T-E/OT, Q1 BSS138, Q2 SI3481DV, X1 DG3XX-02-5.0, Y1 32MHz, Y2 32.768kHz

Commit message: kicad files
Parts:
- added D3: 512-SS24FL, microbuilder:DIODESOD-123
- added U1: MAX5422ETA-T, MAX5422ETA-T:MAX5422ETA-T
Connections:
- new net N$13: C2.P$1, D3.A, L1.2
- net 3.3V: now also U1.VDD
- net BUCK-OUT-1: now also D3.C; no longer C2.P$1, L1.2
- net GND: now also U1.EPAD, U1.GND
Changed lines of the file:
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@@
 <?xml version="1.0" encoding="utf-8"?>
 <!DOCTYPE eagle SYSTEM "eagle.dtd">
-<eagle version="9.5.1">
+<eagle version="9.6.2">
 <drawing>
 <settings>
@@
 <part name="R60" library="microbuilder" deviceset="RESISTOR" device="0603" value="10k"/>
 <part name="IC12" library="SparkFun-RF" deviceset="NRF52832" device=""/>
+<part name="D3" library="microbuilder" deviceset="DIODE" device="SOD-123" value="512-SS24FL"/>
+<part name="U1" library="MAX5422ETA-T" deviceset="MAX5422ETA-T" device=""/>
+<part name="U$5" library="microbuilder" deviceset="3.3V" device=""/>
+<part name="GND19" library="supply1" deviceset="GND" device=""/>
 </parts>
 <sheets>
@@
 512-SS24FL 40V 2A SCHOTTKY</text>
 <wire x1="160.02" y1="134.62" x2="160.02" y2="124.46" width="0.1524" layer="95"/>
-<wire x1="160.02" y1="124.46" x2="175.26" y2="124.46" width="0.1524" layer="95"/>
-<wire x1="175.26" y1="124.46" x2="200.66" y2="124.46" width="0.1524" layer="95"/>
+<wire x1="160.02" y1="124.46" x2="177.8" y2="124.46" width="0.1524" layer="95"/>
+<wire x1="177.8" y1="124.46" x2="200.66" y2="124.46" width="0.1524" layer="95"/>
 <wire x1="200.66" y1="124.46" x2="200.66" y2="134.62" width="0.1524" layer="95"/>
 <wire x1="200.66" y1="134.62" x2="160.02" y2="134.62" width="0.1524" layer="95"/>
-<wire x1="175.26" y1="113.03" x2="175.26" y2="124.46" width="0.1524" layer="95"/>
-<wire x1="173.99" y1="114.3" x2="175.26" y2="113.03" width="0.1524" layer="95"/>
-<wire x1="175.26" y1="113.03" x2="176.53" y2="114.3" width="0.1524" layer="95"/>
+<wire x1="177.8" y1="118.11" x2="177.8" y2="124.46" width="0.1524" layer="95"/>
+<wire x1="176.53" y1="119.38" x2="177.8" y2="118.11" width="0.1524" layer="95"/>
+<wire x1="177.8" y1="118.11" x2="179.07" y2="119.38" width="0.1524" layer="95"/>
 <wire x1="38.1" y1="134.62" x2="38.1" y2="83.82" width="0.1524" layer="95"/>
 <wire x1="38.1" y1="83.82" x2="43.18" y2="83.82" width="0.1524" layer="95"/>
@@
 <attribute name="SHEET" x="230.505" y="5.08" size="2.54" layer="94"/>
 </instance>
+<instance part="D3" gate="G$1" x="177.8" y="111.76" smashed="yes">
+<attribute name="NAME" x="172.72" y="116.84" size="1.27" layer="95"/>
+<attribute name="VALUE" x="172.72" y="114.3" size="1.27" layer="96"/>
+</instance>
+<instance part="U1" gate="A" x="53.34" y="-50.8" smashed="yes">
+<attribute name="NAME" x="40.64" y="-29.48" size="2.0828" layer="95" ratio="10" rot="SR0"/>
+<attribute name="VALUE" x="40.64" y="-75.12" size="2.0828" layer="96" ratio="10" rot="SR0"/>
+</instance>
+<instance part="U$5" gate="G$1" x="73.66" y="-27.94" smashed="yes">
+<attribute name="VALUE" x="72.136" y="-26.924" size="1.27" layer="96"/>
+</instance>
+<instance part="GND19" gate="1" x="73.66" y="-71.12" smashed="yes">
+<attribute name="VALUE" x="71.12" y="-73.66" size="1.778" layer="96"/>
+</instance>
 </instances>
 <busses>
@@
 <pinref part="C6" gate="G$1" pin="P$2"/>
 <pinref part="GND18" gate="1" pin="GND"/>
+</segment>
+<segment>
+<pinref part="U1" gate="A" pin="EPAD"/>
+<pinref part="GND19" gate="1" pin="GND"/>
+<wire x1="71.12" y1="-63.5" x2="73.66" y2="-63.5" width="0.1524" layer="91"/>
+<wire x1="73.66" y1="-63.5" x2="73.66" y2="-66.04" width="0.1524" layer="91"/>
+<pinref part="U1" gate="A" pin="GND"/>
+<wire x1="73.66" y1="-66.04" x2="73.66" y2="-68.58" width="0.1524" layer="91"/>
+<wire x1="71.12" y1="-66.04" x2="73.66" y2="-66.04" width="0.1524" layer="91"/>
+<junction x="73.66" y="-66.04"/>
 </segment>
 </net>
@@
 <pinref part="U$2" gate="G$1" pin="3.3V"/>
 </segment>
+<segment>
+<pinref part="U1" gate="A" pin="VDD"/>
+<pinref part="U$5" gate="G$1" pin="3.3V"/>
+<wire x1="71.12" y1="-33.02" x2="73.66" y2="-33.02" width="0.1524" layer="91"/>
+<wire x1="73.66" y1="-33.02" x2="73.66" y2="-30.48" width="0.1524" layer="91"/>
+</segment>
 </net>
 <net name="PG" class="0">
@@
 <net name="BUCK-OUT-1" class="0">
 <segment>
+<wire x1="185.42" y1="111.76" x2="182.88" y2="111.76" width="0.1524" layer="91"/>
+<pinref part="R7" gate="G$1" pin="2"/>
+<wire x1="182.88" y1="111.76" x2="182.88" y2="121.92" width="0.1524" layer="91"/>
+<wire x1="182.88" y1="121.92" x2="200.66" y2="121.92" width="0.1524" layer="91"/>
+<label x="200.66" y="121.92" size="1.27" layer="95" xref="yes"/>
+<pinref part="D3" gate="G$1" pin="C"/>
+<wire x1="180.34" y1="111.76" x2="182.88" y2="111.76" width="0.1524" layer="91"/>
+<junction x="182.88" y="111.76"/>
+</segment>
+<segment>
+<pinref part="R3" gate="G$1" pin="2"/>
+<wire x1="99.06" y1="25.4" x2="96.52" y2="25.4" width="0.1524" layer="91"/>
+<label x="96.52" y="25.4" size="1.27" layer="95" rot="R180" xref="yes"/>
+</segment>
+</net>
+<net name="N$13" class="0">
+<segment>
 <pinref part="C2" gate="G$1" pin="P$1"/>
 <pinref part="L1" gate="G$1" pin="2"/>
 <wire x1="171.45" y1="111.76" x2="172.72" y2="111.76" width="0.1524" layer="91"/>
+<wire x1="172.72" y1="111.76" x2="172.72" y2="109.22" width="0.1524" layer="91"/>
+<pinref part="D3" gate="G$1" pin="A"/>
+<wire x1="172.72" y1="111.76" x2="175.26" y2="111.76" width="0.1524" layer="91"/>
 <junction x="172.72" y="111.76"/>
-<wire x1="185.42" y1="111.76" x2="177.8" y2="111.76" width="0.1524" layer="91"/>
-<wire x1="177.8" y1="111.76" x2="172.72" y2="111.76" width="0.1524" layer="91"/>
-<wire x1="172.72" y1="111.76" x2="172.72" y2="109.22" width="0.1524" layer="91"/>
-<pinref part="R7" gate="G$1" pin="2"/>
-<wire x1="177.8" y1="111.76" x2="177.8" y2="121.92" width="0.1524" layer="91"/>
-<wire x1="177.8" y1="121.92" x2="200.66" y2="121.92" width="0.1524" layer="91"/>
-<junction x="177.8" y="111.76"/>
-<label x="200.66" y="121.92" size="1.27" layer="95" xref="yes"/>
-</segment>
-<segment>
-<pinref part="R3" gate="G$1" pin="2"/>
-<wire x1="99.06" y1="25.4" x2="96.52" y2="25.4" width="0.1524" layer="91"/>
-<label x="96.52" y="25.4" size="1.27" layer="95" rot="R180" xref="yes"/>
-</segment>
-</net>
+</segment>
+</net>

Commit message: update pcb + test ltspice
Parts:
- removed LED10, LED5, LED6, LED7, LED8, LED9: (no value), microbuilder:LED0805
- removed LED23, LED24: RED, microbuilder:LED0805
- removed LS3: MIC94081YFT-TR, MIC94081YFT-TR:MIC94081YFT-TR
- removed R22, R31, R45, R48, R55, R56, R57, R59: 470, microbuilder:RESISTOR0603
- removed SJ14, SJ15, SJ6, SJ7: JUMPER-SMT_2_NC_TRACE_NO-SILK, SparkFun-Jumpers:JUMPER-SMT_2_NC_TRACE_NO-SILK
- removed SYNC: TPTP09R, testpad:TPTP09R
- added C7: 10u, microbuilder:CAP_CERAMIC0603
- added JP5: JUMPER-SMT_3_NO_NO-SILK, SparkFun-Jumpers:JUMPER-SMT_3_NO_NO-SILK
Connections:
- net P29 renamed MISO
- net P30 renamed MOSI
- net P31 renamed SCK
- removed net N$12: LED9.C, R31.2
- removed net N$19: LED8.C, R55.2
- removed net N$46: LED7.C, R56.2
- removed net N$48: LED6.C, R57.2
- removed net N$49: LED23.C, R45.2
- removed net N$51: LED24.C, R48.2
- removed net N$61: LED5.C, R59.2
- removed net P02: IC12.P0.02/AIN0
- removed net P03: IC12.P0.03/AIN1
- removed net P04: IC12.P0.04/AIN2
- removed net P11: IC12.P0.11, LED5.A
- removed net P12: IC12.P0.12, LED6.A
- removed net P13: IC12.P0.13, LED7.A
- removed net P14: IC12.P0.14, LED8.A
- removed net P17: IC12.P0.17, LED10.A
- removed net UART4_CTS: SJ14.1
- removed net UART4_RTS: SJ15.1
- removed net UART4_RX: SJ7.1
- removed net UART4_TX: SJ6.1
- removed net VDD_BLE_EN: LS3.EN
- new net PWM-CHG: JP5.3
- net 3.3V: no longer JP4.1, LS3.VIN
- net ADC1: now also IC12.P0.02/AIN0
- net BUCK_EN: now also IC12.P0.13
- net EN1: now also IC12.P0.11
- net EN2: now also IC12.P0.12
- net GND: now also C7.P$2, JP5.1; no longer LS3.GND, R12.2, R22.1, R31.1, R55.1, R56.1, R57.1, R59.1
- net LED: now also IC12.P0.17
- net N$6: now also JP5.2, R12.2; no longer LED10.C, R22.2
- net P05: no longer SJ14.2
- net P06: no longer R48.1, SJ7.2
- net P07: no longer SJ15.2
- net P08: no longer R45.1, SJ6.2
- net P15: no longer LED9.A
- net P24: no longer SYNC.TP
- net PG: now also IC12.P0.14
- net V-ICHG: now also IC12.P0.04/AIN2
- net V-VCHG: now also C7.P$1, IC12.P0.03/AIN1
- net VCHG: now also JP4.1
- net VDD_BLE: no longer LED23.A, LED24.A, LS3.VOUT
Other:
- note added: "ADC"
- note removed: "LEDs"
- note removed: "NRF RX"
- note removed: "NRF TX"
- moved on the sheet: C16, D1, D2, R11, R12

Commit message: update pcb
Parts:
- removed U1: MAX5422ETA-T, MAX5422ETA-T:MAX5422ETA-T
- added D4: (no value), diode:DIODE-SOD323-R
- added LS3: MIC94081YFT-TR, MIC94081YFT-TR:MIC94081YFT-TR
- added R16: 47k, microbuilder:RESISTOR0603
Connections:
- net P18 renamed SWO/TDO
- net P26 renamed I2C_SDA
- net P27 renamed I2C_SCL
- removed net P15: IC12.P0.15
- removed net P19: IC12.P0.19
- new net WAKE-UP: D4.C, IC12.P0.19, R16.2
- net 3.3V: no longer U1.VDD
- net GND: now also D4.A, LS3.GND; no longer U1.EPAD, U1.GND
- net LED: now also IC12.P0.15; no longer IC12.P0.17
- net N$10: now also R16.1
- net PWM-CHG: now also IC12.P0.17
- net VDD_BLE: now also LS3.VIN
Other:
- note added: "WAKE UP CHECK???"
- moved on the sheet: X1-1, X1-2
