File: hardware/power-receiving-unit/design1.sch (EAGLE design)
At the start: 77 parts, among them IC12 NRF52832, IC2 STM32L011F3U6TR, IC3 TPS54308DDCR, IC4 MCP6486T-E/OT, Q1 BSS138, Q2 SI3481DV, U1 MAX5422ETA-T, X1 DG3XX-02-5.0, Y1 32MHz, Y2 32.768kHz

Commit message: draft scheme power-receiving-unit
Parts:
- removed C29: 100n, microbuilder:CAP_CERAMIC0603
- removed C62, C63: 6pF, nrf52832-breakout-temp:6PF-0402-50V-0.5%
- removed C64, C65: 15pF, SparkFun-Capacitors:15PF-0402-50V-5%
- removed C66, C68, C69: 0.1uF, SparkFun-Capacitors:0.1UF-0402-16V-10%
- removed C67: 4.7uF, SparkFun-Capacitors:4.7UF0603
- removed C70, C74: DNP, SparkFun-Passives:CAP0402
- removed C71: 1.0uF, SparkFun-Capacitors:1.0UF-0402-16V-10%
- removed C72: 0.8pF, nrf52832-breakout-temp:0.8PF-0402-50V-0.1PF
- removed C73: 100pF, nrf52832-breakout-temp:100PF-0402-50V-5%
- removed C76, C77: 12p, SparkFun-Capacitors:15PF-0402-50V-5%
- removed CRST: 100n, rcl:C-EUC0603
- removed DEBUG: CORTEX_DEBUGPTH, SparkFun-Connectors:CORTEX_DEBUGPTH
- removed IC2: STM32L011F3U6TR, STM32L011F3U6TR:STM32L011F3U6TR
- removed R10, R50: 10k, microbuilder:RESISTOR0603
- removed R13: 100k, microbuilder:RESISTOR0603
- removed U1: MAX5422ETA-T, MAX5422ETA-T:MAX5422ETA-T
- removed UART: (no value), microbuilder:HEADER-1X3ROUND
- removed X1: DG3XX-02-5.0, degson:DG3XX-02-5.0
- removed X2: (no value), adafruit:ANTENNA_U.FL
- added C10, C11, C21, C22, C9: 100n, microbuilder:CAP_CERAMIC0402
- added C14: 1u, microbuilder:CAP_CERAMIC0402
- added C15: 10u, microbuilder:CAP_CERAMIC1206
- added C17, C18: 15p, microbuilder:CAP_CERAMIC0402
- added C19, C20: 6p, microbuilder:CAP_CERAMIC0402
- added C23: DNP, microbuilder:CAP_CERAMIC0402
- added C24: 0.8p, microbuilder:CAP_CERAMIC0402
- added C25, C26: 12p, microbuilder:CAP_CERAMIC0402
- added C8: 4u7, microbuilder:CAP_CERAMIC0603
- added D4: MM3Z3V0T1G, diode:DIODE-SOD323-R
- added D5, D6, D7, D8: PD3S160, diode:PD3S160
- added D9: SMAJ30A, SMAJ30A:SMAJ30A
- added L3, L6: (no value), PowerMagnetics (rev18e):WE-CAIR_4248_744912182
- added LS3: MIC94081YFT-TR, MIC94081YFT-TR:MIC94081YFT-TR
- added R16: 47k, microbuilder:RESISTOR0603
- added SENS: (no value), microbuilder:HEADER-1X4ROUND
- added TP1, TP2: TPTP20SQ, testpad:TPTP20SQ
- added U$18: BLE-ANT, ble-antenna:BLE-ANT
- C12: value 100n -> DNP
- C13: value 100n -> 100p
- JP1: value JUMPER-SMT_3_NO_NO-SILK -> (none); device SparkFun-Jumpers:JUMPER-SMT_3_NO_NO-SILK -> microbuilder:SOLDERJUMPERREFLOW_NOPASTE
- JP3: value JUMPER-SMT_2_NO_NO-SILK -> (none); device SparkFun-Jumpers:JUMPER-SMT_2_NO_NO-SILK -> microbuilder:HEADER-1X2ROUND
- JP4: value JUMPER-SMT_2_NO_NO-SILK -> (none); device SparkFun-Jumpers:JUMPER-SMT_2_NO_NO-SILK -> microbuilder:SOLDERJUMPERREFLOW_NOPASTE
- R49, R60: device microbuilder:RESISTOR0603 -> microbuilder:RESISTOR0402
- R6: value 100k -> 10k; device microbuilder:RESISTOR0603 -> microbuilder:RESISTOR0402
Connections:
- net P18 renamed SWO/TDO
- removed net N$1: JP1.1, R10.1, R13.2
- removed net N$10: Q2.S, R14.1, R8.1, X1-1.KL
- removed net N$11: IC2.PA10, JP3.1
- removed net N$45: C74.1, L2.1, X2.SIGNAL
- removed net N$7: IC3.EN, JP1.2
- removed net NRST: DEBUG.!RESET, IC2.NRST
- removed net P15: IC12.P0.15
- removed net P19: IC12.P0.19
- removed net P20: IC12.P0.20
- removed net P26: C76.2, IC12.P0.26
- removed net P27: IC12.P0.27
- removed net PB9: IC2.PB9, R6.1
- removed net USART2_RX: IC2.PB7, UART.1
- removed net USART2_TX: IC2.PB6, UART.2
- removed net VDD-AUX-EN: IC2.PC14
- new net AGND: C1.P$2, C15.P$2, C16.P$1, C2.P$2, C4.-, C5.P$2, C6.P$2, C7.P$2, D4.A, D6.A, D7.A, D9.A, IC1.GND, IC3.GND, IC4.V-, JP1.1, JP3.2, JP5.1, LS1.GND, LS2.GND, Q1.S, R2.1, R9.2
- new net EN_SENS: IC12.P0.20, LS3.EN
- new net I2C_SCL: IC12.P0.27, SENS.3
- new net I2C_SDA: C25.P$1, IC12.P0.26, SENS.2
- new net MIFA: C23.P$1, L2.1, U$18.1
- new net N$12: L6.1, TP2.TP
- new net N$14: L3.1, TP1.TP
- new net N$15: D5.A, D6.C, L3.2
- new net N$16: D7.C, D8.A, L6.2
- new net VDD_SENS: LS3.VOUT, SENS.1
- new net VDD_WPT: C15.P$1, D5.C, D8.C, D9.C, Q2.S, R14.1, R16.1, R8.1
- new net WAKE-UP: D4.C, IC12.P0.19, R16.2
- net !RESET!: now also C22.P$1; no longer CRST.1
- net 3.3V: no longer U1.VDD
- net ADC1: no longer IC2.PA5, JP3.2
- net ANT: now also C24.P$1; no longer C72.2
- net BUCK_EN: now also IC3.EN; no longer IC2.PA9, JP1.3
- net DEC4: now also C14.P$2; no longer C71.2
- net DEC5: now also C11.P$2; no longer C69.2
- net DEC6: now also C12.P$2; no longer C70.2
- net DEC8: now also C13.P$2; no longer C73.2
- net EN1: no longer IC2.PA0
- net EN2: no longer IC2.PA1
- net GND: now also C10.P$2, C11.P$1, C12.P$1, C13.P$1, C14.P$1, C17.P$2, C18.P$2, C19.P$1, C20.P$1, C21.P$2, C22.P$2, C23.P$2, C24.P$2, C25.P$2, C26.P$2, C8.P$2, C9.P$2, JP1.2, LS3.GND, SENS.4, U$18.2; no longer C1.P$2, C12.P$2, C13.P$2, C16.P$1, C2.P$2, C29.P$2, C4.-, C5.P$2, C6.P$2, C62.1, C63.2, C64.1, C65.1, C66.2, C67.2, C68.2, C69.1, C7.P$2, C70.1, C71.1, C72.1, C73.1, C74.2, C76.1, C77.1, CRST.2, DEBUG.GND@3, DEBUG.GND@5, DEBUG.GNDDTCT, IC1.GND, IC2.VSS, IC3.GND, IC4.V-, JP5.1, LS1.GND, LS2.GND, Q1.S, R10.2, R2.1, R6.2, R9.2, U1.EPAD, U1.GND, UART.3, X1-2.KL, X2.GND@0, X2.GND@1
- net LED: now also IC12.P0.15; no longer IC12.P0.17, IC2.PB1
- net N$50: now also C26.P$1; no longer C77.2
- net P00: now also C17.P$1; no longer C64.2
- net P01: now also C18.P$1; no longer C65.2
- net P16: now also C21.P$1, R6.1; no longer C29.P$1, R50.1
- net PG: no longer IC2.PA4
- net PWM-CHG: now also IC12.P0.17
- net SWDCLK: no longer DEBUG.SWDCLK/TCK, IC2.PA14
- net SWDIO: no longer DEBUG.SWDIO/TMS, IC2.PA13
- net V-ICHG: no longer IC2.PA6
- net V-VCHG: no longer IC2.PA7
- net VCHG: now also JP3.1; no longer C12.P$1, C13.P$1, DEBUG.VCC, IC2.VDD, IC2.VDDA
- net VDD_BLE: now also C10.P$1, C8.P$1, C9.P$1, LS3.VIN, R6.2; no longer C66.1, C67.1, C68.1, R50.2
- net VIN: no longer R13.1
- net XC1: now also C20.P$2; no longer C62.2
- net XC2: now also C19.P$2; no longer C63.1
Other:
- note added: "50V"
- note added: "WAKE UP CHECK???"
- note added: "https://www.infineon.com/dgdl/Infineon-AN91445_Antenna_Design_and_RF_Layout_Guidelines-ApplicationNotes-v09_00-EN.pdf"
- note removed: "Add boot button"
- note removed: "These pin could be used for: - informing application MCU, energy storage is charging - informing application MCU, energy storage is fully charger by small pulse"

Commit message: power receiving unit PCB V1.0 ready
Parts:
- added C27, C28, C29: 100n, microbuilder:CAP_CERAMIC0402
- added JP10, JP11, JP12, JP13, JP14, JP6, JP7, JP8, JP9: JUMPER-SMT_2_NO_NO-SILK, SparkFun-Jumpers:JUMPER-SMT_2_NO_NO-SILK
- renumbered SENS to SENSOR
Connections:
- new net P02: C27.P$1, IC12.P0.02/AIN0, JP12.1
- new net P03: C28.P$1, IC12.P0.03/AIN1, JP13.1
- new net P04: C29.P$1, IC12.P0.04/AIN2, JP14.1
- new net P11: IC12.P0.11, JP6.1
- new net P12: IC12.P0.12, JP7.1
- new net P13: IC12.P0.13, JP8.1
- new net P14: IC12.P0.14, JP9.1
- new net P17: IC12.P0.17, JP10.1
- new net P19: IC12.P0.19, JP11.1
- net ADC1: now also JP12.2; no longer IC12.P0.02/AIN0
- net BUCK_EN: now also JP8.2; no longer IC12.P0.13
- net EN1: now also JP6.2; no longer IC12.P0.11
- net EN2: now also JP7.2; no longer IC12.P0.12
- net GND: now also C27.P$2, C28.P$2, C29.P$2
- net PG: now also JP9.2; no longer IC12.P0.14
- net PWM-CHG: now also JP10.2; no longer IC12.P0.17
- net V-ICHG: now also JP14.2; no longer IC12.P0.04/AIN2
- net V-VCHG: now also JP13.2; no longer IC12.P0.03/AIN1
- net WAKE-UP: now also JP11.2; no longer IC12.P0.19
Other:
- note removed: "WAKE UP CHECK???"
- moved on the sheet: LED1, R1
