File: hardware/power-receiving-unit/design1.brd (EAGLE design)
At the start: 55 x 40 mm, 107 parts, among them IC3 TPS54308DDCR, IC4 MCP6486T-E/OT, Q1 BSS138, Q2 SI3481DV, Q3 PMDPB55XP, Q4 DMG1012T, Q5 DMG1012T, Y1 32MHz, Y2 32.768kHz

Commit message: Update firmware - hardware all
Parts:
- C23: value 0.8p -> 1.2p
- D1, D2: value SDM03U40 -> RB751S40T1G
- IC1: value (none) -> AP7381-33SA-7
- IC5: value (none) -> TPL0401A-10DCKR
Changed lines of the file:
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@@
 <attribute name="VALUE" x="29.6545" y="28.7655" size="0.4064" layer="27" font="vector" ratio="10" rot="R90"/>
 </element>
-<element name="D1" library="microbuilder" package="SOD-523" value="SDM03U40" x="23.1775" y="24.13" smashed="yes" rot="R90">
+<element name="D1" library="microbuilder" package="SOD-523" value="RB751S40T1G" x="23.1775" y="24.13" smashed="yes" rot="R90">
 <attribute name="NAME" x="20.32" y="22.38375" size="0.6096" layer="25" font="vector"/>
 <attribute name="VALUE" x="23.9015" y="24.846" size="0.4064" layer="27" ratio="10" rot="R90"/>
 </element>
-<element name="D2" library="microbuilder" package="SOD-523" value="SDM03U40" x="23.1775" y="22.86" smashed="yes" rot="R90">
+<element name="D2" library="microbuilder" package="SOD-523" value="RB751S40T1G" x="23.1775" y="22.86" smashed="yes" rot="R90">
 <attribute name="NAME" x="20.32" y="21.59" size="0.6096" layer="25" font="vector"/>
 <attribute name="VALUE" x="23.9015" y="23.576" size="0.4064" layer="27" ratio="10" rot="R90"/>
@@
 <attribute name="VALUE" x="50.673" y="24.79675" size="0.4064" layer="27" font="vector" ratio="10"/>
 </element>
-<element name="IC1" library="microbuilder" package="SOT23-R" value="" x="32.7025" y="36.195" smashed="yes" rot="R180">
+<element name="IC1" library="microbuilder" package="SOT23-R" value="AP7381-33SA-7" x="32.7025" y="36.195" smashed="yes" rot="R180">
 <attribute name="NAME" x="31.75" y="38.1" size="0.6096" layer="25" font="vector"/>
 <attribute name="VALUE" x="30.9245" y="36.83" size="0.4064" layer="27" ratio="10" rot="R180"/>
@@
 <attribute name="VALUE" x="32.280225" y="2.314575" size="0.4064" layer="27" ratio="10" rot="R180"/>
 </element>
-<element name="C23" library="microbuilder" package="0402" value="0.8p" x="43.815" y="13.97" smashed="yes" rot="R90">
+<element name="C23" library="microbuilder" package="0402" value="1.2p" x="43.815" y="13.97" smashed="yes" rot="R90">
 <attribute name="NAME" x="43.33875" y="12.54125" size="0.6096" layer="25" font="vector" rot="R270"/>
 <attribute name="VALUE" x="44.45" y="15.367" size="0.4064" layer="27" ratio="10" rot="R90"/>
@@
 <attribute name="VALUE" x="47.33925" y="20.5105" size="0.4064" layer="27" font="vector" ratio="10"/>
 </element>
-<element name="IC5" library="TPL0401A-10DCKR" package="SOT65P210X110-6N" value="" x="20.32" y="24.4475" smashed="yes">
+<element name="IC5" library="TPL0401A-10DCKR" package="SOT65P210X110-6N" value="TPL0401A-10DCKR" x="20.32" y="24.4475" smashed="yes">
 <attribute name="AVAILABILITY" value="In Stock" x="20.32" y="24.4475" size="1.778" layer="27" display="off"/>
 <attribute name="CHECK_PRICES" value="https://www.snapeda.com/parts/TPL0401A-10DCKR/Texas+Instruments/view-part/?ref=eda" x="20.32" y="24.4475" size="1.778" layer="27" display="off"/>
