File: hardware/power-transmitting-unit/eagle-archive/design1.sch (EAGLE design)
At the start: 54 parts, among them IC1 LM5113SDX/NOPB, IC2 AP7381-50Y-13, IC3 DSC1001DI2-006.7800, IC4 AP7381-33Y-13, IC5 74LVC1G00GW, IC6 74LVC1G08GW, J1 62201021121, U1 ADS1115IDGST

Commit message: Update HW PTU
Parts:
- removed C18, C21, C22: 100n, microbuilder:CAP_CERAMIC0603
- removed C19, C20: 10u, microbuilder:CAP_CERAMIC0603
- removed C23: (no value), Kondensatoren (rev17a):WCAP-CSGP_0805_885012207103_WAVE
- removed D5, D6: SDM03U40, microbuilder:DIODESOD-523
- removed IC3: DSC1001DI2-006.7800, DSC1001:DSC1001DI2-006.7800
- removed IC4: AP7381-33Y-13, AP7381:AP7381-50Y-13
- removed IC5: 74LVC1G00GW, 74LVC1G00GW:74LVC1G00GW
- removed IC6: 74LVC1G08GW, 74LVC1G00GW:74LVC1G00GW
- removed J1: 62201021121, Eagle_WR-PHD (rev22a):6220XX21121_62201021121
- removed L3: (no value), PowerMagnetics (rev18e):WE-DD_1280_744873150
- removed R4, R5, R6: 180, microbuilder:RESISTOR0402
- removed TP5: TPTP20SQ, testpad:TPTP20SQ
- removed U1: ADS1115IDGST, ADS1115IDGST:ADS1115IDGST
- removed VR1: XL6009, XL6009:XL6009
- added L2: (no value), PowerMagnetics (rev18e):WE-DD_1260_CROSSED_744871100
- C14, C15, C16: value 10n -> (none)
Connections:
- removed net +3V3: C18.P$1, C19.P$1, IC3.VDD, IC4.VOUT, J1.5
- removed net N$2: D5.C, IC5.Y, R4.1
- removed net N$4: D6.C, IC6.Y, R5.1
- removed net OOK: IC5.A, IC6.A, R6.2, TP5.TP
- removed net OSC: IC5.B, IC6.B
- removed net OSC_CLK: IC3.OUT
- removed net OSC_ENABLE: IC3.!SHDN!
- removed net SCL: J1.9
- removed net SDA: J1.10
- net +5V: no longer C21.P$1, C22.P$1, IC5.VCC, IC6.VCC, J1.6, R6.1
- net AGND: no longer C18.P$2, C19.P$2, C20.P$2, C21.P$2, C22.P$2, IC3.GND, IC4.GND, IC5.GND, IC6.GND, J1.3, J1.7, J1.8, L3.1, VR1.GND
- net HSIG: no longer D5.A, R4.2
- net LSIG: no longer D6.A, R5.2
- net UAV_BAT: no longer C20.P$1, IC4.VIN
- net VAMP: no longer J1.1, J1.2, J1.4
Other:
- note removed: "3V3 MCU + OSC"
- note removed: "AND"
- note removed: "Gates & Dead time control"
- note removed: "NAND"
- note removed: "Oscillator"
- moved on the sheet: C3, C4, IC2, TP3, TP4
