File: hardware/power-transmitting-unit/PSU-board/design.brd (EAGLE design)
At the start: 30 x 30 mm, 58 parts, among them IC10 TSC1031, IC2 AP7381-50Y-13, IC4 AP7381-33Y-13, IC7 TSC1031, IC8 TSC1031, J2 62201021121, U1 ADS1115IDGST

Commit message: Update hardware PTU
Parts:
- removed C23: 1u, Kondensatoren (rev17a):WCAP-CSGP_0805_WAVE
- removed C24: 10u, microbuilder:0805
- removed C25, C26: 100 µF, Eagle_WCAP-ASNP (rev20a):WCAP-ASNP_8X10.5(DXL)
- removed D7: SS34, microbuilder:SOD-123
- removed L2: 2u2, EMCComponents (rev19b):WE-LQS_3015
- removed L3: (no value), PowerMagnetics (rev18e):WE-DD_1260/1280
- removed R13: 39k, microbuilder:0603
- removed SJ5, SJ6: (no value), microbuilder:SOLDERJUMPER_REFLOW
- removed TP3, TP4, TP6, TP7: TPTP20SQ, testpad:TP20SQ
- removed U1: ADS1115IDGST, ADS1115IDGST:SOP50P490X110-10N
- removed VR1: XL6009, XL6009:DPAK170P1435X465-6N
- added C1: 1u, Kondensatoren (rev17a):WCAP-CSGP_0805_WAVE
- added C10, C11, C12, C13, C8, C9: 10u, microbuilder:1206
- added C2: 10u, microbuilder:0805
- added C5: 100n, microbuilder:0402
- added C7: 1u, microbuilder:0603
- added D1: SS34, microbuilder:SOD-123
- added IC1: TPL0401A-10DCKR, TPL0401A-10DCKR:SOT65P210X110-6N
- added IC3: LT8330, LT8330ES6TR:TSOT-23_S6
- added IC5: ADS1115IDGST, ADS1115IDGST:SOP50P490X110-10N
- added L1: 744877100, PowerMagnetics (rev18e):WE-DD_7345
- added L4: 2u2, EMCComponents (rev19b):WE-LQS_3015
- added L7: 742792692, PowerMagnetics (rev18e):WE-CBF_0603(W=2.2)
- added R1: 10k, microbuilder:0603
- added R2: 1k, microbuilder:0603
- added SJ7: SOLDERJUMPERNO, SparkFun-Retired:SJ_2S-NO
- added SJ8: (no value), SparkFun-Retired:SJ_3
- added U2, U3: (no value), UAV-connector:HOLE
- C27, C57, R10, R11, R12, R17, R28, R30, R31, R33, R9: device microbuilder:0603 -> microbuilder:0402
- moved R8 119.0 mm to (45.4, 2.54), turned to 90 degrees
- moved R16 117.6 mm to (50.2, 7.62), turned to 270 degrees
- moved R7 112.9 mm to (43.5, 2.54), turned to 90 degrees
- moved R12 110.1 mm to (47.6, 6.67)
- moved C52 105.8 mm to (40.4, 9.53), turned to 90 degrees
- moved R34 105.1 mm to (33.7, 13.0), turned to 270 degrees
- moved J2 102.0 mm to (50.0, 3.00)
- moved C55 100.5 mm to (27.3, 8.57), turned to 90 degrees
- moved C30 100.2 mm to (45.5, 7.63), turned to 90 degrees
- moved IC2 97.8 mm to (36.2, 3.81)
- moved C57 97.7 mm to (36.8, 12.7), turned to 90 degrees
- moved IC8 89.6 mm to (43.8, 9.46), flipped to the bottom
- moved SJ1 89.6 mm to (22.5, 8.89), flipped to the bottom
- moved C4 89.0 mm to (40.6, 2.70), turned to 90 degrees
- moved C28 88.6 mm to (30.5, 9.21), turned to 270 degrees
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Connections:
- removed net 3.3V: C52.1, C56.1, IC10.5, IC8.5
- removed net N$10: C25.1, D7.C, L2.1
- removed net N$9: C23.2, L3.3
- removed net SCL: J2.9
- removed net SDA: J2.10
- removed net VAMP_EN: VR1.2
- new net N$1: IC3.1, L1.4
- new net N$16: IC1.6, R2.2, SJ7.1
- new net N$2: C1.2, L1.3
- new net N$4: C27.1, IC5.8, L7.2
- new net N$6: C1.1, D1.A, L1.2
- new net N$7: C11.1, C12.1, C13.1, D1.C, L4.1, R1.2
- new net N$8: IC3.4, SJ8.2
- new net SEPIC_FB: IC1.5, IC3.3, R1.1, SJ7.2
- net +3V3: now also C52.1, C56.1, IC1.1, IC10.5, IC8.5, L7.1; no longer C27.1, U1.8
- net AGND: now also C10.2, C11.2, C12.2, C13.2, C2.2, C5.2, C7.2, C8.2, C9.2, IC1.2, IC3.2, IC5.1, IC5.3, L1.1, R2.1, SJ8.1, U2.2, U3.2; no longer C24.2, C25.2, C26.2, L3.1, TP4.TP, TP7.TP, U1.1, U1.3, VR1.1
- net AIN0: now also IC5.4; no longer U1.4
- net AIN1: now also IC5.5; no longer U1.5
- net AIN2: now also IC5.6; no longer U1.6
- net AIN3: now also IC5.7; no longer U1.7
- net I2C_SCL: now also IC1.3, IC5.10, J2.9, R7.2; no longer U1.10
- net I2C_SDA: now also IC1.4, IC5.9, J2.10; no longer R7.2, U1.9
- net N$5: now also C7.1, IC3.5; no longer C23.1, D7.A, L3.4
- net UAV_BAT: now also U2.1; no longer R30.2, R32.1, SJ5.1, TP3.TP
- net UAV_BAT_1: now also R30.2, R32.1, SJ8.3, U3.1; no longer TP6.TP
- net VAMP: no longer SJ6.2
- net V_SEPIC_IN: now also C10.1, C8.1, C9.1, IC3.6; no longer C26.1, L3.2, SJ5.2, VR1.3, VR1.4, VR1.6
- net V_SEPIC_OUT: now also C2.1, L4.2; no longer C24.1, L2.2, SJ6.1
Routing:
- net +3V3: track 0.00 -> 85.0 mm, vias 0 -> 5
- net I2C_SDA: track 0.00 -> 49.3 mm, vias 0 -> 3
- net I2C_SCL: track 0.00 -> 47.5 mm, vias 0 -> 4
- net +5V: track 0.00 -> 35.0 mm, vias 0 -> 3
- net N$7: track 0.00 -> 24.2 mm, vias 0 -> 1
- net UAV_BAT: track 0.00 -> 21.2 mm, vias 0 -> 11
- net AIN2: track 0.00 -> 17.5 mm, vias 0 -> 2
- net UAV_BAT_1: track 0.00 -> 17.0 mm, vias 0 -> 5
- net N$8: track 0.00 -> 15.1 mm, vias 0 -> 2
- net AIN3: track 0.00 -> 12.8 mm, vias 0 -> 1
- net N$27: track 0.00 -> 11.7 mm
- net V_SEPIC_IN: track 0.00 -> 11.3 mm
- net AIN0: track 0.00 -> 10.7 mm
- net SEPIC_FB: track 0.00 -> 10.1 mm, vias 0 -> 1
- net N$30: track 0.00 -> 9.66 mm
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- added copper zone on layer 1, net AGND
- added copper zone on layer 16, net AGND
- added copper zone on layer 1, net N$1
- added copper zone on layer 1, net UAV_BAT
- added copper zone on layer 16, net UAV_BAT
- added copper zone on layer 1, net UAV_BAT_1
- added copper zone on layer 16, net UAV_BAT_1
- added copper zone on layer 1, net VAMP
- added copper zone on layer 1, net V_SEPIC_OUT
Other:
- board size 30 x 30 mm -> 61 x 35 mm
- board text added: "EN"
- board text added: "GND"
- board text added: "Jarne Van Mulders"
- board text added: "NR013"
- board text added: "V+"
