File: hardware/power-transmitting-unit/PSU-board/design.sch (EAGLE design)
At the start: 58 parts, among them IC10 TSC1031, IC2 AP7381-50Y-13, IC4 AP7381-33Y-13, IC7 TSC1031, IC8 TSC1031, J2 62201021121, U1 ADS1115IDGST

Commit message: Update hardware PTU
Parts:
- removed C23: 1u, Kondensatoren (rev17a):WCAP-CSGP_0805_885012207103_WAVE
- removed C24: 10u, microbuilder:CAP_CERAMIC0805
- removed C25, C26: 100 µF, Eagle_WCAP-ASNP (rev20a):WCAP-ASNP_8X10.5_865250453009
- removed D7: SS34, microbuilder:DIODESOD-123
- removed L2: 2u2, EMCComponents (rev19b):WE-LQS_3015_74404032022
- removed L3: (no value), PowerMagnetics (rev18e):WE-DD_1280_744873150
- removed R13: 39k, microbuilder:RESISTOR0603
- removed SJ5, SJ6: (no value), microbuilder:SOLDERJUMPERREFLOW
- removed TP3, TP4, TP6, TP7: TPTP20SQ, testpad:TPTP20SQ
- removed U1: ADS1115IDGST, ADS1115IDGST:ADS1115IDGST
- removed VR1: XL6009, XL6009:XL6009
- added C1: 1u, Kondensatoren (rev17a):WCAP-CSGP_0805_885012207103_WAVE
- added C10, C11, C12, C13, C8, C9: 10u, microbuilder:CAP_CERAMIC1206
- added C2: 10u, microbuilder:CAP_CERAMIC0805
- added C5: 100n, microbuilder:CAP_CERAMIC0402
- added C7: 1u, microbuilder:CAP_CERAMIC0603
- added D1: SS34, microbuilder:DIODESOD-123
- added IC1: TPL0401A-10DCKR, TPL0401A-10DCKR:TPL0401A-10DCKR
- added IC3: LT8330, LT8330ES6TR:LT8330ES6TR
- added IC5: ADS1115IDGST, ADS1115IDGST:ADS1115IDGST
- added L1: 744877100, PowerMagnetics (rev18e):WE-DD_7345_744877100
- added L4: 2u2, EMCComponents (rev19b):WE-LQS_3015_74404032022
- added L7: 742792692, PowerMagnetics (rev18e):WE-CBF_0603_742792692_WB_HS
- added R1: 10k, microbuilder:RESISTOR0603
- added R2: 1k, microbuilder:RESISTOR0603
- added SJ7: SOLDERJUMPERNO, SparkFun-Retired:SOLDERJUMPERNO
- added SJ8: (no value), SparkFun-Retired:SOLDERJUMPER_2WAYS
- added U2, U3: (no value), UAV-connector:UAV-CONNECT
- C27, C57: device microbuilder:CAP_CERAMIC0603 -> microbuilder:CAP_CERAMIC0402
- R10, R11, R12, R17, R28, R30, R31, R33, R9: device microbuilder:RESISTOR0603 -> microbuilder:RESISTOR0402
Connections:
- removed net 3.3V: C52.P$1, C56.P$1, IC10.VCC+, IC8.VCC+
- removed net N$10: C25.1, D7.C, L2.1
- removed net N$9: C23.2, L3.3
- removed net SCL: J2.9
- removed net SDA: J2.10
- removed net VAMP_EN: VR1.EN
- new net N$1: IC3.SW, L1.4
- new net N$16: IC1.H, R2.2, SJ7.1
- new net N$2: C1.2, L1.3
- new net N$4: C27.P$1, IC5.VDD, L7.2
- new net N$6: C1.1, D1.A, L1.2
- new net N$7: C11.P$1, C12.P$1, C13.P$1, D1.C, L4.1, R1.2
- new net N$8: IC3.EN/UVLO, SJ8.2
- new net SEPIC_FB: IC1.W, IC3.FBX, R1.1, SJ7.2
- net +3V3: now also C52.P$1, C56.P$1, IC1.VDD, IC10.VCC+, IC8.VCC+, L7.1; no longer C27.P$1, U1.VDD
- net AGND: now also C10.P$2, C11.P$2, C12.P$2, C13.P$2, C2.P$2, C5.P$2, C7.P$2, C8.P$2, C9.P$2, IC1.GND, IC3.GND, IC5.ADDR, IC5.GND, L1.1, R2.1, SJ8.1, U2.GND, U3.GND; no longer C24.P$2, C25.2, C26.2, L3.1, TP4.TP, TP7.TP, U1.ADDR, U1.GND, VR1.GND
- net AIN0: now also IC5.AIN0; no longer U1.AIN0
- net AIN1: now also IC5.AIN1; no longer U1.AIN1
- net AIN2: now also IC5.AIN2; no longer U1.AIN2
- net AIN3: now also IC5.AIN3; no longer U1.AIN3
- net I2C_SCL: now also IC1.SCL, IC5.SCL, J2.9, R7.2; no longer U1.SCL
- net I2C_SDA: now also IC1.SDA, IC5.SDA, J2.10; no longer R7.2, U1.SDA
- net N$5: now also C7.P$1, IC3.INTVCC; no longer C23.1, D7.A, L3.2
- net UAV_BAT: now also U2.V+; no longer R30.2, R32.1, SJ5.1, TP3.TP
- net UAV_BAT_1: now also R30.2, R32.1, SJ8.3, U3.V+; no longer TP6.TP
- net VAMP: no longer SJ6.2
- net V_SEPIC_IN: now also C10.P$1, C8.P$1, C9.P$1, IC3.VIN; no longer C26.1, L3.4, SJ5.2, VR1.SW, VR1.VIN
- net V_SEPIC_OUT: now also C2.P$1, L4.2; no longer C24.P$1, L2.2, SJ6.1
Other:
- note removed: "50V"
- note removed: "digi pot"

Commit message: Update PTU firmware and hardware
Other:
- note added: "I2C ADDR 0x2E"
- note added: "I2C ADDR 0x48"
Changed lines of the file:
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@@
 <setting verticaltext="up"/>
 </settings>
-<grid distance="0.1" unitdist="inch" unit="inch" style="lines" multiple="1" display="yes" altdistance="0.01" altunitdist="inch" altunit="inch"/>
+<grid distance="0.1" unitdist="inch" unit="inch" style="lines" multiple="1" display="no" altdistance="0.01" altunitdist="inch" altunit="inch"/>
 <layers>
 <layer number="1" name="Top" color="4" fill="1" visible="no" active="no"/>
@@
 PCA9570GMH</text>
 <text x="6.35" y="6.35" size="6.4516" layer="95">DRAMCO</text>
+<text x="137.16" y="124.46" size="1.778" layer="95">I2C ADDR 0x2E</text>
 </plain>
 <instances>
@@
 <text x="165.1" y="132.08" size="1.778" layer="95">SEPIC current</text>
 <text x="6.35" y="6.35" size="6.4516" layer="95">DRAMCO</text>
+<text x="203.2" y="71.12" size="1.778" layer="95">I2C ADDR 0x48</text>
+<text x="203.2" y="71.12" size="1.778" layer="95">I2C ADDR 0x48</text>
 </plain>
 <instances>
