File: hardware/power-transmitting-unit/design1.brd (EAGLE design)
At the start: 56.2 x 54 mm, 120 parts, among them IC1 LM5113SDX/NOPB, IC12 NRF52832, IC2 AP7381-50Y-13, IC3 DSC1001DI2-006.7800, IC4 AP7381-33Y-13, IC5 74LVC1G00GW, IC6 74LVC1G08GW, IC7 MCP6486T-E/OT, J1 62201021121, J2 62201021121, U1 ADS1115IDGST, Y1 32MHz, Y2 32.768kHz

Commit message: Update SW PRU & HW PRU + PTU
Parts:
- added C51, C52, C55, C56: 100n, microbuilder:0402
- added C57: 100n, microbuilder:0603
- added IC10, IC8: TSC1031, TSC1031:SOP65P640X120-8N
- added R16, R27, R29, R32: 0.01, microbuilder:0805
- added R17, R28, R33: 1k, microbuilder:0603
- added R18, R19, R30, R31: 100, microbuilder:0603
- added R25, R26: (no value), microbuilder:0603
- added R34: 100k, microbuilder:0603
- added R35: 10k, microbuilder:0603
- added SJ1, SJ2, SJ3: SOLDERJUMPERTRACE, SparkFun-Retired:SJ_2S-TRACE
- added TP6, TP7: TPTP20SQ, testpad:TP20SQ
- IC7: value MCP6486T-E/OT -> TSC1031; device SparkFun-Retired:SOT23-5 -> TSC1031:SOP65P640X120-8N
- R10, R11: value 1k -> 100
- R12, R9: value 39k -> 100
- moved IC12 203.6 mm to (18.8, 11.2)
- moved R12 188.3 mm to (-119.8, -320.5)
- moved R9 188.3 mm to (-120.5, -323.0)
- moved C30 186.0 mm to (-126.5, -325.5)
- moved IC7 121.3 mm to (-120.2, -245.2)
- moved C29 103.0 mm to (-123.2, -240.2)
- moved J1 79.3 mm to (19.2, 3.00)
- moved TP4 32.1 mm to (-12.1, 8.67)
- moved TP3 31.3 mm to (-7.35, 6.68)
Connections:
- net N$16 renamed AIN1
- removed net BUCK-OUT-1: R10.2
- removed net BUCK-OUT-2: R11.2
- removed net N$17: U1.6
- removed net N$18: U1.7
- new net AIN0: C57.1, R34.1, R35.2, U1.4
- new net AIN2: IC10.4, U1.6
- new net AIN3: IC8.4, U1.7
- new net N$14: R18.1, R19.2
- new net N$24: R25.1, R26.2
- new net N$25: IC7.3, SJ1.2
- new net N$26: C29.1, IC7.1, R11.1
- new net N$27: C29.2, IC7.8, R10.1
- new net N$29: C51.1, IC10.1, R31.1
- new net N$30: C51.2, IC10.8, R30.1
- new net N$31: IC7.2, R28.1
- new net N$32: IC10.3, SJ2.2
- new net N$33: IC10.2, R33.1
- new net UAV_BAT_1: R11.2, R27.2, R29.2, TP6.TP
- new net VOUT_AIN0: IC7.4
- new net V_SEPIC_IN: C26.1, L3.2, R31.2, R32.2, VR1.3, VR1.4, VR1.6
- new net V_SEPIC_OUT: C24.1, L2.2, R16.1, R9.2
- net +5V: now also C55.1, IC7.5
- net 3.3V: now also C52.1, C56.1, IC10.5, IC8.5; no longer C29.1, IC7.5
- net AGND: now also C52.2, C55.2, C56.2, C57.2, IC10.6, IC10.7, IC7.6, IC7.7, IC8.6, IC8.7, R17.2, R19.1, R26.1, R28.2, R33.2, R35.1, SJ1.1, SJ2.1, SJ3.1, TP7.TP; no longer C29.2, IC7.2, R9.1
- net N$11: now also C30.2, IC8.8, R9.1; no longer C24.1, L2.2
- net N$12: now also IC8.3, SJ3.2; no longer C30.1, IC7.4, R11.1, R12.1
- net N$13: now also IC8.2, R17.1; no longer C30.2, IC7.3, R10.1, R9.2
- net N$15: now also R18.2; no longer U1.4
- net N$3: now also C30.1, IC8.1, R12.1; no longer C26.1, L3.2, VR1.3, VR1.4, VR1.6
- net UAV_BAT: now also R10.2, R27.1, R29.1, R30.2, R32.1, R34.2
- net V-ICHG: no longer IC7.1, R12.2
- net VAMP: now also R12.2, R16.2, R25.2

Commit message: Update hardware PTU
Parts:
- removed C19, C20, C28, C3, C4: 10u, microbuilder:0603
- removed C23: 1u, Kondensatoren (rev17a):WCAP-CSGP_0805_WAVE
- removed C24: 10u, microbuilder:0805
- removed C25, C26: 100 µF, Eagle_WCAP-ASNP (rev20a):WCAP-ASNP_8X10.5(DXL)
- removed C27, C57: 100n, microbuilder:0603
- removed C29, C30, C51, C52, C55, C56: 100n, microbuilder:0402
- removed C38, C39: 15p, microbuilder:0402
- removed D7: SS34, microbuilder:SOD-123
- removed IC10, IC7, IC8: TSC1031, TSC1031:SOP65P640X120-8N
- removed IC12: NRF52832, SparkFun-RF:QFN48-6X6MM
- removed IC4: AP7381-33Y-13, AP7381:FOOT_XC6201P332PR-G
- removed L2: 2u2, EMCComponents (rev19b):WE-LQS_3015
- removed L3: (no value), PowerMagnetics (rev18e):WE-DD_1260/1280
- removed L5: 10uH, microbuilder:_0603MP
- removed L6: 15nH, nrf52832-breakout-temp:0402
- removed R10, R11, R12, R18, R19, R30, R31, R9: 100, microbuilder:0603
- removed R13: 39k, microbuilder:0603
- removed R16, R27, R29, R32: 0.01, microbuilder:0805
- removed R17, R28, R33: 1k, microbuilder:0603
- removed R34: 100k, microbuilder:0603
- removed R35: 10k, microbuilder:0603
- removed R7, R8: 4k7, microbuilder:0603
- removed SENSOR, UART_INTERFACE: (no value), microbuilder:1X04_ROUND
- removed SJ2, SJ3: SOLDERJUMPERTRACE, SparkFun-Retired:SJ_2S-TRACE
- removed TP3, TP4, TP6, TP7: TPTP20SQ, testpad:TP20SQ
- removed U$48: BLE-ANT, ble-antenna:ANT-2G4
- removed U1: ADS1115IDGST, ADS1115IDGST:SOP50P490X110-10N
- removed VR1: XL6009, XL6009:DPAK170P1435X465-6N
- removed Y2: 32.768kHz, SparkFun-Clocks:CRYSTAL-SMD-3.2X1.5MM
- C1, C2, C6, C7, R1, R2: device microbuilder:0603 -> microbuilder:0402
- D2, D3, D5, D6: value SDM03U40 -> RB751S40T1G
- FET3: value (none) -> EPC2038
- IC2: value AP7381-50Y-13 -> NRF52832; device AP7381:FOOT_XC6201P332PR-G -> SparkFun-RF:QFN48-6X6MM-EXTENDED
- J2: value 62201021121 -> 636101111001; device Eagle_WR-PHD (rev22a):62201021121 -> Eagle_WR-UMRF (rev21b):636101111001
- JP1: device microbuilder:SOLDERJUMPER_REFLOW_NOPASTE -> microbuilder:1X03_ROUND
- R25: value (none) -> 100k
- R26: value (none) -> 10k
- SJ1: value SOLDERJUMPERTRACE -> SOLDERJUMPERNO; device SparkFun-Retired:SJ_2S-TRACE -> SparkFun-Retired:SJ_2S-NO
- moved SJ1 338.3 mm to (-25.8, 61.8)
- moved R26 300.7 mm to (27.2, 2.50), flipped to the bottom, turned to 90 degrees
- moved R25 297.8 mm to (25.8, 2.50), flipped to the bottom, turned to 270 degrees
- moved C40 251.2 mm to (23.8, 16.2), flipped to the bottom, turned to 90 degrees
- moved C41 249.1 mm to (25.2, 16.2), flipped to the bottom, turned to 90 degrees
- moved C35 245.6 mm to (22.0, 16.5), turned to 270 degrees
- moved C34 244.4 mm to (14.8, 16.5), turned to 270 degrees
- moved C36 241.9 mm to (20.8, 16.5), turned to 270 degrees
- moved R49 239.7 mm to (11.5, 6.25), turned to 180 degrees
- moved L4 239.5 mm to (25.0, 11.0), turned to 180 degrees
- moved C44 237.5 mm to (27.0, 11.8), turned to 90 degrees
- moved C37 237.2 mm to (17.2, 16.5), turned to 270 degrees
- moved Y1 236.8 mm to (24.5, 16.2)
- moved C45 232.6 mm to (23.0, 11.8), turned to 90 degrees
- moved C31 232.1 mm to (15.8, 16.8), turned to 90 degrees
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Connections:
- net BUCK_EN renamed N$10
- net EN2 renamed N$9
- net PG renamed N$11
- net PWM-CHG renamed N$12
- net V-ICHG renamed N$16
- net V-VCHG renamed N$15
- net WAKE-UP renamed N$13
- removed net 3.3V: C52.1, C56.1, IC10.5, IC8.5
- removed net ADC1: JP12.2
- removed net AIN0: C57.1, R34.1, R35.2, U1.4
- removed net AIN1: U1.5
- removed net AIN2: IC10.4, U1.6
- removed net AIN3: IC8.4, U1.7
- removed net EN1: JP6.2
- removed net MIFA: C44.1, L4.1, U$48.1
- removed net N$10 (its old number): C25.1, D7.C, L2.1
- removed net N$11 (its old number): C30.2, IC8.8, R9.1
- removed net N$12 (its old number): IC8.3, SJ3.2
- removed net N$13 (its old number): IC8.2, R17.1
- removed net N$14: R18.1, R19.2
- removed net N$15 (its old number): R18.2
- removed net N$24: R25.1, R26.2
- removed net N$25: IC7.3, SJ1.2
- removed net N$26: C29.1, IC7.1, R11.1
- removed net N$27: C29.2, IC7.8, R10.1
- removed net N$29: C51.1, IC10.1, R31.1
- removed net N$30: C51.2, IC10.8, R30.1
- removed net N$31: IC7.2, R28.1
- removed net N$32: IC10.3, SJ2.2
- removed net N$33: IC10.2, R33.1
- removed net N$5: C23.1, D7.A, L3.4
- removed net N$53: L5.2, L6.1
- removed net N$9 (its old number): C23.2, L3.3
- removed net UAV_BAT: C20.1, C4.1, IC2.3, IC4.3, R10.2, R27.1, R29.1, R30.2, R32.1, R34.2, TP3.TP
- removed net UAV_BAT_1: R11.2, R27.2, R29.2, TP6.TP
- removed net VAMP_EN: VR1.2
- removed net VCHG: JP4.1
- removed net VDD_SENS: LS3.1, SENSOR.1
- removed net VOUT_AIN0: IC7.4
- removed net V_SEPIC_IN: C26.1, L3.2, R31.2, R32.2, VR1.3, VR1.4, VR1.6
- removed net V_SEPIC_OUT: C24.1, L2.2, R16.1, R9.2
- new net UFL: C44.1, J2.1, L4.1
- new net V-VAMP: JP12.2, R25.1, R26.2
- net !RESET!: now also IC2.24; no longer IC12.24
- net +3V3: now also JP4.1; no longer C19.1, C27.1, C28.1, IC4.1, J2.5, R7.1, R8.1, U1.8
- net +5V: no longer C3.1, C55.1, IC2.1, IC7.5, J2.6
- net AGND: no longer C19.2, C20.2, C24.2, C25.2, C26.2, C27.2, C28.2, C3.2, C4.2, C52.2, C55.2, C56.2, C57.2, IC10.6, IC10.7, IC2.2, IC2.2.1, IC4.2, IC4.2.1, IC7.6, IC7.7, IC8.6, IC8.7, J2.3, J2.7, J2.8, JP1.1, L3.1, R17.2, R19.1, R28.2, R33.2, R35.1, SJ1.1, SJ2.1, SJ3.1, TP4.TP, TP7.TP, U1.1, U1.3, VR1.1
- net ANT: now also IC2.30; no longer IC12.30
- net DCC: now also IC2.47; no longer IC12.47, L5.1
- net DEC4: now also IC2.46; no longer IC12.46, L6.2
- net DEC5: now also IC2.1; no longer IC12.1
- net DEC6: now also IC2.32; no longer IC12.32
- net DEC8: now also IC2.33; no longer IC12.33
- net EN_SENS: now also IC2.23; no longer IC12.23, LS3.4
- net GND: now also IC2.31, IC2.45, IC2.EP, J2.2, J2.3, JP1.3; no longer C38.2, C39.2, IC12.31, IC12.45, IC12.EP, JP1.2, SENSOR.4, U$48.2
- net I2C_SCL: now also IC2.39; no longer IC12.39, SENSOR.3, U1.10
- net I2C_SDA: now also IC2.38; no longer IC12.38, R7.2, R8.2, SENSOR.2, U1.9
- net LED: now also IC2.18; no longer IC12.18
- net MISO: now also IC2.41; no longer IC12.41
- net MOSI: now also IC2.42; no longer IC12.42
- net N$3: now also IC3.1, SJ1.2; no longer C30.1, IC8.1, R12.1
- net N$50: now also IC2.37; no longer IC12.37
- net NC: now also IC2.44; no longer IC12.44
- net OSC_ENABLE: now also JP6.2, SJ1.1; no longer IC3.1
- net P00: now also IC2.2; no longer C38.1, IC12.2, Y2.P$2
- net P01: now also IC2.3; no longer C39.1, IC12.3, Y2.P$1
- net P02: now also IC2.4; no longer IC12.4
- net P03: now also IC2.5; no longer IC12.5
- net P04: now also IC2.6; no longer IC12.6
- net P05: now also IC2.7; no longer IC12.7, UART_INTERFACE.3
- net P06: now also IC2.8, JP1.2; no longer IC12.8, UART_INTERFACE.2
- net P07: now also IC2.9; no longer IC12.9, UART_INTERFACE.4
- net P08: now also IC2.10, JP1.1; no longer IC12.10, UART_INTERFACE.1
- net P09: now also IC2.11; no longer IC12.11
- net P10: now also IC2.12; no longer IC12.12
- net P11: now also IC2.14; no longer IC12.14
- net P12: now also IC2.15; no longer IC12.15
- net P13: now also IC2.16; no longer IC12.16
- net P14: now also IC2.17; no longer IC12.17
- net P16: now also IC2.19; no longer IC12.19
- net P17: now also IC2.20; no longer IC12.20
- net P19: now also IC2.22; no longer IC12.22
- net P22: now also IC2.27; no longer IC12.27
- net P23: now also IC2.28; no longer IC12.28
- net P24: now also IC2.29; no longer IC12.29
- net P28: now also IC2.40; no longer IC12.40
- net SCK: now also IC2.43; no longer IC12.43
- net SCL: no longer J2.9
- net SDA: no longer J2.10
- net SWDCLK: now also IC2.25; no longer IC12.25
- net SWDIO: now also IC2.26; no longer IC12.26
- net SWO/TDO: now also IC2.21; no longer IC12.21
- net VAMP: no longer J2.1, J2.2, J2.4, R12.2, R16.2
- net VDD_BLE: now also IC2.13, IC2.36, IC2.48; no longer IC12.13, IC12.36, IC12.48, LS3.3
- net XC1: now also IC2.34; no longer IC12.34
- net XC2: now also IC2.35; no longer IC12.35

Commit message: Update PTU firmware and hardware
Parts:
- removed C42, C48, C49, C50: 100n, microbuilder:0402
- removed C46, C47: 12p, microbuilder:0402
- removed JP10, JP11, JP12, JP13, JP14, JP6, JP7, JP8, JP9: JUMPER-SMT_2_NO_NO-SILK, SparkFun-Jumpers:SMT-JUMPER_2_NO_NO-SILK
- removed JP4: (no value), microbuilder:SOLDERJUMPER_REFLOW_NOPASTE
- removed LS3: MIC94081YFT-TR, MIC94081YFT-TR:IC_MIC94081YFT-TR
- removed R15: 10k, microbuilder:0402
- removed R25: 100k, microbuilder:0603
- removed R26: 10k, microbuilder:0603
- removed UPDATE: (no value), Eagle_SWITCHES (rev18c):434111043826
- added C3, C4: 100n, microbuilder:0402
- added L2: 742792692, PowerMagnetics (rev18e):WE-CBF_0603(W=2.2)
- added POWER: JUMPER-SMT_2_NO_NO-SILK, SparkFun-Jumpers:SMT-JUMPER_2_NO_NO-SILK
- added R10: 100k, microbuilder:0402
- added R7, R8, R9: 10k, microbuilder:0402
- added TP10, TP11, TP12, TP4, TP6, TP7, TP9: TPTP10SQ, testpad:TP10SQ
- added TP3, TP8: TPTP20SQ, testpad:TP20SQ
- C21, C22, C5, C8, C9, R3: device microbuilder:0603 -> microbuilder:0402
- TP5: value TPTP20SQ -> TPTP10SQ; device testpad:TP20SQ -> testpad:TP10SQ
- moved SJ1 64.2 mm to (24.5, 21.8), turned to 180 degrees
- moved R60 63.3 mm to (11.8, 15.8), turned to 270 degrees
- moved IC3 60.4 mm to (22.0, 21.8), turned to 180 degrees
- moved C8 59.8 mm to (21.2, 33.0), flipped to the bottom, turned to 270 degrees
- moved FET3 59.7 mm to (22.8, 33.8), flipped to the bottom
- moved C18 57.1 mm to (19.8, 21.8), turned to 90 degrees
- moved R3 54.9 mm to (21.2, 35.8), flipped to the bottom, turned to 90 degrees
- moved C9 52.7 mm to (22.8, 35.8), flipped to the bottom, turned to 90 degrees
- moved C43 50.6 mm to (10.2, 15.8), turned to 90 degrees
- moved D4 50.1 mm to (22.0, 37.2), flipped to the bottom, turned to 180 degrees
- moved TP5 34.1 mm to (21.5, 27.5)
- moved R6 33.4 mm to (19.8, 26.8)
- moved IC5 32.9 mm to (12.2, 26.8)
- moved C21 32.7 mm to (12.2, 26.8)
- moved C22 32.0 mm to (16.2, 26.8)
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Connections:
- removed net N$10: JP8.2
- removed net N$11: JP9.2
- removed net N$12: JP10.2
- removed net N$13: JP11.2
- removed net N$15: JP13.2
- removed net N$16: JP14.2
- removed net N$50: C47.1, IC2.37
- removed net N$6: FET2.3, FET2.5, FET2.6
- removed net N$9: JP7.2
- removed net OSC: IC5.1, IC6.1
- removed net P02: C48.1, IC2.4, JP12.1
- removed net P03: C49.1, IC2.5, JP13.1
- removed net P04: C50.1, IC2.6, JP14.1
- removed net P11: IC2.14, JP6.1
- new net N$14: L2.1, POWER.2
- new net P25: IC2.37
- new net V-5V: C3.1, IC2.6, R7.2, R8.1
- net +3V3: now also POWER.1, TP6.TP; no longer JP4.1
- net +5V: now also R8.2, TP4.TP
- net AGND: now also FET2.3, FET2.5, FET2.6, R9.1, TP7.TP, TP8.TP; no longer R26.1
- net GND: now also C3.2, C4.2, R7.1; no longer C42.2, C46.2, C47.2, C48.2, C49.2, C50.2, LS3.2, UPDATE.1
- net I2C_SDA: no longer C46.1
- net OSC_CLK: now also IC5.1, IC6.1
- net OSC_ENABLE: now also IC2.14; no longer JP6.2
- net P12: now also TP9.TP; no longer JP7.1
- net P13: now also TP10.TP; no longer JP8.1
- net P14: now also TP11.TP; no longer JP9.1
- net P16: no longer C42.1, R15.1, UPDATE.2
- net P17: now also TP12.TP; no longer JP10.1
- net P19: no longer JP11.1
- net V-VAMP: now also C4.1, IC2.4, R10.1, R9.2; no longer JP12.2, R25.1, R26.2
- net VAMP: now also R10.2, TP3.TP; no longer R25.2
- net VDD_BLE: now also IC2.5, L2.2; no longer JP4.2, R15.2
Other:
- board text added: "+3V3"
- board text added: "+5V"
- board text added: "GND"
- board text added: "OOK"
- board text added: "Power Transmitting Unit"
- board text added: "V1.0"
- board text added: "VAMP"
