File: hardware/power-transmitting-unit/design1.sch (EAGLE design)
At the start: 34 parts, among them IC1 LM5113SDX/NOPB, IC2 AP7381-50Y-13

Commit message: ltspice buck-boost
Parts:
- added L2: (no value), PowerMagnetics (rev18e):WE-DD_1260_CROSSED_744871100
Other:
- note added: "Input voltage will vary during flight"
- note added: "approx. 10 - 16.8 V"
Changed lines of the file:
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@@
 <part name="TP4" library="testpad" library_urn="urn:adsk.eagle:library:385" deviceset="TP" device="TP20SQ" package3d_urn="urn:adsk.eagle:package:27980/1"/>
 <part name="U$21" library="SparkFun-PowerSymbols" deviceset="AGND" device=""/>
+<part name="L2" library="PowerMagnetics (rev18e)" deviceset="WE-DD_1260_CROSSED" device="" technology="_744871100"/>
 </parts>
 <sheets>
@@
 <wire x1="55.88" y1="63.5" x2="55.88" y2="99.06" width="0.1524" layer="95" style="shortdash"/>
 <text x="-40.64" y="96.52" size="1.27" layer="95">buck (boost) converter</text>
+<text x="-185.42" y="53.34" size="1.27" layer="95">Input voltage will vary during flight</text>
+<text x="-185.42" y="50.8" size="1.27" layer="95">approx. 10 - 16.8 V</text>
 </plain>
 <instances>
@@
 <attribute name="VALUE" x="-157.48" y="40.386" size="1.778" layer="96" align="top-center"/>
 </instance>
+<instance part="L2" gate="G$1" x="7.62" y="78.74" smashed="yes">
+<attribute name="NAME" x="2.88" y="82.25" size="1.778" layer="95"/>
+<attribute name="VALUE" x="3.18" y="73.62" size="1.778" layer="96"/>
+</instance>
 </instances>

Commit message: Update HW PTU
Parts:
- added C18, C21, C22, C27: 100n, microbuilder:CAP_CERAMIC0603
- added C19, C20, C28: 10u, microbuilder:CAP_CERAMIC0603
- added C23: 1u, Kondensatoren (rev17a):WCAP-CSGP_0805_885012207103_WAVE
- added C24: 10u, microbuilder:CAP_CERAMIC0805
- added C25, C26: 100 µF, Eagle_WCAP-ASNP (rev20a):WCAP-ASNP_8X10.5_865250453009
- added C29, C30, C32, C33, C34, C42, C43, C48, C49, C50: 100n, microbuilder:CAP_CERAMIC0402
- added C31: 4u7, microbuilder:CAP_CERAMIC0603
- added C35, C44: DNP, microbuilder:CAP_CERAMIC0402
- added C36: 100p, microbuilder:CAP_CERAMIC0402
- added C37: 1u, microbuilder:CAP_CERAMIC0402
- added C38, C39: 15p, microbuilder:CAP_CERAMIC0402
- added C40, C41: 6p, microbuilder:CAP_CERAMIC0402
- added C45: 0.8p, microbuilder:CAP_CERAMIC0402
- added C46, C47: 12p, microbuilder:CAP_CERAMIC0402
- added D5, D6: SDM03U40, microbuilder:DIODESOD-523
- added D7: SS34, microbuilder:DIODESOD-123
- added DEBUG1: CORTEX_DEBUGPTH, SparkFun-Connectors:CORTEX_DEBUGPTH
- added IC12: NRF52832, SparkFun-RF:NRF52832
- added IC3: DSC1001DI2-006.7800, DSC1001:DSC1001DI2-006.7800
- added IC4: AP7381-33Y-13, AP7381:AP7381-50Y-13
- added IC5: 74LVC1G00GW, 74LVC1G00GW:74LVC1G00GW
- added IC6: 74LVC1G08GW, 74LVC1G00GW:74LVC1G00GW
- added IC7: MCP6486T-E/OT, SparkFun-Retired:MCP6291T-E/OT
- added J1, J2: 62201021121, Eagle_WR-PHD (rev22a):6220XX21121_62201021121
- added JP1, JP4: (no value), microbuilder:SOLDERJUMPERREFLOW_NOPASTE
- added JP10, JP11, JP12, JP13, JP14, JP6, JP7, JP8, JP9: JUMPER-SMT_2_NO_NO-SILK, SparkFun-Jumpers:JUMPER-SMT_2_NO_NO-SILK
- added L3: (no value), PowerMagnetics (rev18e):WE-DD_1280_744873150
- added L4: 3.9nH, nrf52832-breakout-temp:INDUCTOR-0402-3.9NH
- added L5: 10uH, microbuilder:INDUCTOR_0603MP
- added L6: 15nH, nrf52832-breakout-temp:INDUCTOR-0402-3.9NH
- added LED1: (no value), microbuilder:LED0805
- added LS3: MIC94081YFT-TR, MIC94081YFT-TR:MIC94081YFT-TR
- added R10, R11: 1k, microbuilder:RESISTOR0603
- added R12, R13, R9: 39k, microbuilder:RESISTOR0603
- added R14: 220, microbuilder:RESISTOR0603
- added R15, R49, R60: 10k, microbuilder:RESISTOR0402
- added R4, R5, R6: 180, microbuilder:RESISTOR0402
- added R7, R8: 4k7, microbuilder:RESISTOR0603
- added SENSOR, UART_INTERFACE: (no value), microbuilder:HEADER-1X4ROUND
- added TP5: TPTP20SQ, testpad:TPTP20SQ
- added U$48: BLE-ANT, ble-antenna:BLE-ANT
- added U1: ADS1115IDGST, ADS1115IDGST:ADS1115IDGST
- added UPDATE: (no value), Eagle_SWITCHES (rev18c):434111043826
- added VR1: XL6009, XL6009:XL6009
- added Y1: 32MHz, nrf52832-breakout-temp:CRYSTAL-32MHZ-SMD-2.0X1.6MM
- added Y2: 32.768kHz, SparkFun-Clocks:CRYSTAL-32.768KHZSMD-3.2X1.5
- C14, C15, C16: value (none) -> 10n
- L2: value (none) -> 2u2; device PowerMagnetics (rev18e):WE-DD_1260_CROSSED_744871100 -> EMCComponents (rev19b):WE-LQS_3015_74404032022
Connections:
- new net !RESET!: C43.P$1, DEBUG1.!RESET, IC12.P0.21/RESET, R60.2
- new net +3V3: C18.P$1, C19.P$1, C27.P$1, C28.P$1, IC3.VDD, IC4.VOUT, J1.5, J2.5, R7.1, R8.1, U1.VDD
- new net 3.3V: C29.P$1, IC7.V+
- new net ADC1: JP12.2
- new net ANT: C45.P$1, IC12.ANT, L4.2
- new net BUCK-OUT-1: R10.2
- new net BUCK-OUT-2: R11.2
- new net BUCK_EN: JP8.2
- new net DCC: IC12.DCC, L5.1
- new net DEC4: C37.P$2, IC12.DEC4, L6.2
- new net DEC5: C34.P$2, IC12.DEC1
- new net DEC6: C35.P$2, IC12.DEC2
- new net DEC8: C36.P$2, IC12.DEC3
- new net EN1: JP6.2
- new net EN2: JP7.2
- new net EN_SENS: IC12.P0.20, LS3.EN
- new net GND: C31.P$2, C32.P$2, C33.P$2, C34.P$1, C35.P$1, C36.P$1, C37.P$1, C38.P$2, C39.P$2, C40.P$1, C41.P$1, C42.P$2, C43.P$2, C44.P$2, C45.P$2, C46.P$2, C47.P$2, C48.P$2, C49.P$2, C50.P$2, DEBUG1.GND@3, DEBUG1.GND@5, DEBUG1.GNDDTCT, IC12.VSS, JP1.2, LED1.C, LS3.GND, R49.1, SENSOR.4, U$48.2, UPDATE.1
- new net I2C_SCL: IC12.P0.27, SENSOR.3, U1.SCL
- new net I2C_SDA: C46.P$1, IC12.P0.26, R7.2, R8.2, SENSOR.2, U1.SDA
- new net LED: IC12.P0.15, R14.2
- new net MIFA: C44.P$1, L4.1, U$48.1
- new net MISO: IC12.P0.29/AIN5
- new net MOSI: IC12.P0.30/AIN6
- new net N$10: C25.1, D7.C, L2.1
- new net N$11: C24.P$1, L2.2
- new net N$12: C30.P$1, IC7.-IN, R11.1, R12.1
- new net N$13: C30.P$2, IC7.+IN, R10.1, R9.2
- new net N$15: U1.AIN0
- new net N$16: U1.AIN1
- new net N$17: U1.AIN2
- new net N$18: U1.AIN3
- new net N$2: D5.C, IC5.Y, R4.1
- new net N$20: LED1.A, R14.1
- new net N$3: C26.1, L3.4, VR1.SW, VR1.VIN
- new net N$4: D6.C, IC6.Y, R5.1
- new net N$5: C23.1, D7.A, L3.2
- new net N$50: C47.P$1, IC12.P0.25
- new net N$53: L5.2, L6.1
- new net N$9: C23.2, L3.3
- new net NC: IC12.NC
- new net OOK: IC5.A, IC6.A, R6.2, TP5.TP
- new net OSC: IC5.B, IC6.B
- new net OSC_CLK: IC3.OUT
- new net OSC_ENABLE: IC3.!SHDN!
- new net P00: C38.P$1, IC12.P0.00/XL1, Y2.2
- new net P01: C39.P$1, IC12.P0.01/XL2, Y2.1
- new net P02: C48.P$1, IC12.P0.02/AIN0, JP12.1
- new net P03: C49.P$1, IC12.P0.03/AIN1, JP13.1
- new net P04: C50.P$1, IC12.P0.04/AIN2, JP14.1
- new net P05: IC12.P0.05/AIN3, UART_INTERFACE.3
- new net P06: IC12.P0.06, UART_INTERFACE.2
- new net P07: IC12.P0.07, UART_INTERFACE.4
- new net P08: IC12.P0.08, UART_INTERFACE.1
- new net P09: IC12.P0.09/NFC1
- new net P10: IC12.P0.10/NFC2
- new net P11: IC12.P0.11, JP6.1
- new net P12: IC12.P0.12, JP7.1
- new net P13: IC12.P0.13, JP8.1
- new net P14: IC12.P0.14, JP9.1
- new net P16: C42.P$1, IC12.P0.16, R15.1, UPDATE.2
- new net P17: IC12.P0.17, JP10.1
- new net P19: IC12.P0.19, JP11.1
- new net P22: IC12.P0.22
- new net P23: IC12.P0.23
- new net P24: IC12.P0.24
- new net P28: IC12.P0.28/AIN4
- new net PG: JP9.2
- new net PWM-CHG: JP10.2
- new net SCK: IC12.P0.31/AIN7
- new net SCL: J1.9, J2.9
- new net SDA: J1.10, J2.10
- new net SWDCLK: DEBUG1.SWDCLK/TCK, IC12.SWDCLK, R49.2
- new net SWDIO: DEBUG1.SWDIO/TMS, IC12.SWDIO
- new net SWO/TDO: DEBUG1.SWO/TDO, IC12.P0.18
- new net V-ICHG: IC7.OUT, JP14.2, R12.2
- new net V-VCHG: JP13.2
- new net VAMP_EN: VR1.EN
- new net VCHG: JP4.1
- new net VDD_BLE: C31.P$1, C32.P$1, C33.P$1, DEBUG1.VCC, IC12.VDD, JP4.2, LS3.VIN, R15.2, R60.1
- new net VDD_SENS: LS3.VOUT, SENSOR.1
- new net WAKE-UP: JP11.2
- new net XC1: C41.P$2, IC12.XC1(32MHZ), Y1.2
- new net XC2: C40.P$2, IC12.XC2(32MHZ), Y1.1
- net +5V: now also C21.P$1, C22.P$1, IC5.VCC, IC6.VCC, J1.6, J2.6, R6.1
- net AGND: now also C18.P$2, C19.P$2, C20.P$2, C21.P$2, C22.P$2, C24.P$2, C25.2, C26.2, C27.P$2, C28.P$2, C29.P$2, IC3.GND, IC4.GND, IC5.GND, IC6.GND, IC7.V-, J1.3, J1.7, J1.8, J2.3, J2.7, J2.8, JP1.1, L3.1, R9.1, U1.ADDR, U1.GND, VR1.GND
- net HSIG: now also D5.A, R4.2
- net LSIG: now also D6.A, R5.2
- net UAV_BAT: now also C20.P$1, IC4.VIN
- net VAMP: now also J1.1, J1.2, J1.4, J2.1, J2.2, J2.4
Other:
- note added: "32.768kHz Crystal (RTC)"
- note added: "3V3 MCU + OSC"
- note added: "50V"
- note added: "ADC"
- note added: "AND"
- note added: "Add DC/DC converter as power supply for nRF52 nRF will automatically switch between DC/DC and LDO to ensure minimal power consumption"
- note added: "Application note, filter shunt resistor (current measurements). https://www.st.com/resource/en/application_note/an4304-how-to-filter-the-input-of-a-highside-current-sensing-stmicroelectronics.pdf"
- note added: "BT Module"
- note added: "Button"
- note added: "CTS"
- note added: "Cortex Debug Connector"
- note added: "DRAMCO"
- note added: "Gates & Dead time control"
- note added: "I2C ADC"
- note added: "IO EXPANDER REQUIRED? PCA9570GMH"
- note added: "Jarne Van Mulders"
- note added: "MOUSER: 609-L-07C15NKV6T"
- note added: "MOUSER: 81-LQM18FN100M00D"
- note added: "NAND"
- note added: "NRF52832 (BLE INTERFACE)"
- note added: "NRF52832 CTS"
- note added: "NRF52832 RTS"
- note added: "NRF52832 RXI"
- note added: "NRF52832 TXI"
- note added: "Oscillator"
- note added: "Pin 13"
- note added: "Pin 36"
- note added: "Pin 48"
- note added: "RTS"
- note added: "RX"
- note added: "Supply Decoupling"
- note added: "TX"
- note added: "UART CONNECTION"
- note added: "add pull-down to swd-clk to prevent entering debug mode"
- note added: "digi pot"
- note added: "https://www.infineon.com/dgdl/Infineon-AN91445_Antenna_Design_and_RF_Layout_Guidelines-ApplicationNotes-v09_00-EN.pdf"
- note added: "nRF52832"
- note added: "nRF52832 Supply Range !1.7 - 3.6V DC!"
- moved on the sheet: C3, C4, IC2, TP3, TP4

Commit message: Update SW PRU & HW PRU + PTU
Parts:
- added C51, C52, C55, C56: 100n, microbuilder:CAP_CERAMIC0402
- added C57: 100n, microbuilder:CAP_CERAMIC0603
- added IC10, IC8: TSC1031, TSC1031:TSC1031IPT
- added R16, R27, R29, R32: 0.01, microbuilder:RESISTOR0805
- added R17, R28, R33: 1k, microbuilder:RESISTOR0603
- added R18, R19, R30, R31: 100, microbuilder:RESISTOR0603
- added R25, R26: (no value), microbuilder:RESISTOR0603
- added R34: 100k, microbuilder:RESISTOR0603
- added R35: 10k, microbuilder:RESISTOR0603
- added SJ1, SJ2, SJ3: SOLDERJUMPERTRACE, SparkFun-Retired:SOLDERJUMPERTRACE
- added TP6, TP7: TPTP20SQ, testpad:TPTP20SQ
- IC7: value MCP6486T-E/OT -> TSC1031; device SparkFun-Retired:MCP6291T-E/OT -> TSC1031:TSC1031IPT
- R10, R11: value 1k -> 100
- R12, R9: value 39k -> 100
Connections:
- net N$16 renamed AIN1
- removed net BUCK-OUT-1: R10.2
- removed net BUCK-OUT-2: R11.2
- removed net N$17: U1.AIN2
- removed net N$18: U1.AIN3
- new net AIN0: C57.P$1, R34.1, R35.2, U1.AIN0
- new net AIN2: IC10.VOUT, U1.AIN2
- new net AIN3: IC8.VOUT, U1.AIN3
- new net N$14: R18.1, R19.2
- new net N$24: R25.1, R26.2
- new net N$25: IC7.SEL, SJ1.2
- new net N$26: C29.P$1, IC7.VM, R11.1
- new net N$27: C29.P$2, IC7.VP, R10.1
- new net N$29: C51.P$1, IC10.VM, R31.1
- new net N$30: C51.P$2, IC10.VP, R30.1
- new net N$31: IC7.A1, R28.1
- new net N$32: IC10.SEL, SJ2.2
- new net N$33: IC10.A1, R33.1
- new net UAV_BAT_1: R11.2, R27.2, R29.2, TP6.TP
- new net VOUT_AIN0: IC7.VOUT
- new net V_SEPIC_IN: C26.1, L3.4, R31.2, R32.2, VR1.SW, VR1.VIN
- new net V_SEPIC_OUT: C24.P$1, L2.2, R16.1, R9.2
- net +5V: now also C55.P$1, IC7.VCC+
- net 3.3V: now also C52.P$1, C56.P$1, IC10.VCC+, IC8.VCC+; no longer C29.P$1, IC7.V+
- net AGND: now also C52.P$2, C55.P$2, C56.P$2, C57.P$2, IC10.GND, IC10.VCC-, IC7.GND, IC7.VCC-, IC8.GND, IC8.VCC-, R17.2, R19.1, R26.1, R28.2, R33.2, R35.1, SJ1.1, SJ2.1, SJ3.1, TP7.TP; no longer C29.P$2, IC7.V-, R9.1
- net N$11: now also C30.P$2, IC8.VP, R9.1; no longer C24.P$1, L2.2
- net N$12: now also IC8.SEL, SJ3.2; no longer C30.P$1, IC7.-IN, R11.1, R12.1
- net N$13: now also IC8.A1, R17.1; no longer C30.P$2, IC7.+IN, R10.1, R9.2
- net N$15: now also R18.2; no longer U1.AIN0
- net N$3: now also C30.P$1, IC8.VM, R12.1; no longer C26.1, L3.4, VR1.SW, VR1.VIN
- net UAV_BAT: now also R10.2, R27.1, R29.1, R30.2, R32.1, R34.2
- net V-ICHG: no longer IC7.OUT, R12.2
- net VAMP: now also R12.2, R16.2, R25.2
Other:
- note added: "Amplification 50V/V"
- note added: "BETAFLIGHT current"
- note added: "CONNECT WITH NRF"
- note added: "FSR = ±2.048 V"
- note added: "Resistor values should be equal!"
- note added: "SEPIC current"
- note added: "Sense Amplifier"
- moved on the sheet: C19, C20, C23, C24, C25, C26, C27, C28, C29, C3, C30, C4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

Commit message: Update hardware PTU
Parts:
- removed C19, C20, C28, C3, C4: 10u, microbuilder:CAP_CERAMIC0603
- removed C23: 1u, Kondensatoren (rev17a):WCAP-CSGP_0805_885012207103_WAVE
- removed C24: 10u, microbuilder:CAP_CERAMIC0805
- removed C25, C26: 100 µF, Eagle_WCAP-ASNP (rev20a):WCAP-ASNP_8X10.5_865250453009
- removed C27, C57: 100n, microbuilder:CAP_CERAMIC0603
- removed C29, C30, C51, C52, C55, C56: 100n, microbuilder:CAP_CERAMIC0402
- removed C38, C39: 15p, microbuilder:CAP_CERAMIC0402
- removed D7: SS34, microbuilder:DIODESOD-123
- removed IC10, IC7, IC8: TSC1031, TSC1031:TSC1031IPT
- removed IC12: NRF52832, SparkFun-RF:NRF52832
- removed IC4: AP7381-33Y-13, AP7381:AP7381-50Y-13
- removed L2: 2u2, EMCComponents (rev19b):WE-LQS_3015_74404032022
- removed L3: (no value), PowerMagnetics (rev18e):WE-DD_1280_744873150
- removed L5: 10uH, microbuilder:INDUCTOR_0603MP
- removed L6: 15nH, nrf52832-breakout-temp:INDUCTOR-0402-3.9NH
- removed R10, R11, R12, R18, R19, R30, R31, R9: 100, microbuilder:RESISTOR0603
- removed R13: 39k, microbuilder:RESISTOR0603
- removed R16, R27, R29, R32: 0.01, microbuilder:RESISTOR0805
- removed R17, R28, R33: 1k, microbuilder:RESISTOR0603
- removed R34: 100k, microbuilder:RESISTOR0603
- removed R35: 10k, microbuilder:RESISTOR0603
- removed R7, R8: 4k7, microbuilder:RESISTOR0603
- removed SENSOR, UART_INTERFACE: (no value), microbuilder:HEADER-1X4ROUND
- removed SJ2, SJ3: SOLDERJUMPERTRACE, SparkFun-Retired:SOLDERJUMPERTRACE
- removed TP3, TP4, TP6, TP7: TPTP20SQ, testpad:TPTP20SQ
- removed U$48: BLE-ANT, ble-antenna:BLE-ANT
- removed U1: ADS1115IDGST, ADS1115IDGST:ADS1115IDGST
- removed VR1: XL6009, XL6009:XL6009
- removed Y2: 32.768kHz, SparkFun-Clocks:CRYSTAL-32.768KHZSMD-3.2X1.5
- C1, C2, C6, C7: device microbuilder:CAP_CERAMIC0603 -> microbuilder:CAP_CERAMIC0402
- D2, D3, D5, D6: value SDM03U40 -> RB751S40T1G
- FET3: value (none) -> EPC2038
- IC2: value AP7381-50Y-13 -> NRF52832; device AP7381:AP7381-50Y-13 -> SparkFun-RF:NRF52832-EXTENDED
- J2: value 62201021121 -> 636101111001; device Eagle_WR-PHD (rev22a):6220XX21121_62201021121 -> Eagle_WR-UMRF (rev21b):636101111001
- JP1: device microbuilder:SOLDERJUMPERREFLOW_NOPASTE -> microbuilder:HEADER-1X3ROUND
- R1, R2: device microbuilder:RESISTOR0603 -> microbuilder:RESISTOR0402
- R25: value (none) -> 100k
- R26: value (none) -> 10k
- SJ1: value SOLDERJUMPERTRACE -> SOLDERJUMPERNO; device SparkFun-Retired:SOLDERJUMPERTRACE -> SparkFun-Retired:SOLDERJUMPERNO
Connections:
- net BUCK_EN renamed N$10
- net EN2 renamed N$9
- net PG renamed N$11
- net PWM-CHG renamed N$12
- net V-ICHG renamed N$16
- net V-VCHG renamed N$15
- net WAKE-UP renamed N$13
- removed net 3.3V: C52.P$1, C56.P$1, IC10.VCC+, IC8.VCC+
- removed net ADC1: JP12.2
- removed net AIN0: C57.P$1, R34.1, R35.2, U1.AIN0
- removed net AIN1: U1.AIN1
- removed net AIN2: IC10.VOUT, U1.AIN2
- removed net AIN3: IC8.VOUT, U1.AIN3
- removed net EN1: JP6.2
- removed net MIFA: C44.P$1, L4.1, U$48.1
- removed net N$10 (its old number): C25.1, D7.C, L2.1
- removed net N$11 (its old number): C30.P$2, IC8.VP, R9.1
- removed net N$12 (its old number): IC8.SEL, SJ3.2
- removed net N$13 (its old number): IC8.A1, R17.1
- removed net N$14: R18.1, R19.2
- removed net N$15 (its old number): R18.2
- removed net N$24: R25.1, R26.2
- removed net N$25: IC7.SEL, SJ1.2
- removed net N$26: C29.P$1, IC7.VM, R11.1
- removed net N$27: C29.P$2, IC7.VP, R10.1
- removed net N$29: C51.P$1, IC10.VM, R31.1
- removed net N$30: C51.P$2, IC10.VP, R30.1
- removed net N$31: IC7.A1, R28.1
- removed net N$32: IC10.SEL, SJ2.2
- removed net N$33: IC10.A1, R33.1
- removed net N$5: C23.1, D7.A, L3.2
- removed net N$53: L5.2, L6.1
- removed net N$9 (its old number): C23.2, L3.3
- removed net UAV_BAT: C20.P$1, C4.P$1, IC2.VIN, IC4.VIN, R10.2, R27.1, R29.1, R30.2, R32.1, R34.2, TP3.TP
- removed net UAV_BAT_1: R11.2, R27.2, R29.2, TP6.TP
- removed net VAMP_EN: VR1.EN
- removed net VCHG: JP4.1
- removed net VDD_SENS: LS3.VOUT, SENSOR.1
- removed net VOUT_AIN0: IC7.VOUT
- removed net V_SEPIC_IN: C26.1, L3.4, R31.2, R32.2, VR1.SW, VR1.VIN
- removed net V_SEPIC_OUT: C24.P$1, L2.2, R16.1, R9.2
- new net UFL: C44.P$1, J2.1, L4.1
- new net V-VAMP: JP12.2, R25.1, R26.2
- net !RESET!: now also IC2.P0.21/RESET; no longer IC12.P0.21/RESET
- net +3V3: now also JP4.1; no longer C19.P$1, C27.P$1, C28.P$1, IC4.VOUT, J2.5, R7.1, R8.1, U1.VDD
- net +5V: now also FET3.S; no longer C3.P$1, C55.P$1, FET3.SOURCE, IC2.VOUT, IC7.VCC+, J2.6
- net AGND: now also FET2.SR; no longer C19.P$2, C20.P$2, C24.P$2, C25.2, C26.2, C27.P$2, C28.P$2, C3.P$2, C4.P$2, C52.P$2, C55.P$2, C56.P$2, C57.P$2, FET2.SOURCE-RETURN, IC10.GND, IC10.VCC-, IC2.GND, IC4.GND, IC7.GND, IC7.VCC-, IC8.GND, IC8.VCC-, J2.3, J2.7, J2.8, JP1.1, L3.1, R17.2, R19.1, R28.2, R33.2, R35.1, SJ1.1, SJ2.1, SJ3.1, TP4.TP, TP7.TP, U1.ADDR, U1.GND, VR1.GND
- net ANT: now also IC2.ANT; no longer IC12.ANT
- net DCC: now also IC2.DCC; no longer IC12.DCC, L5.1
- net DEC4: now also IC2.DEC4; no longer IC12.DEC4, L6.2
- net DEC5: now also IC2.DEC1; no longer IC12.DEC1
- net DEC6: now also IC2.DEC2; no longer IC12.DEC2
- net DEC8: now also IC2.DEC3; no longer IC12.DEC3
- net EN_SENS: now also IC2.P0.20; no longer IC12.P0.20, LS3.EN
- net GBTST: now also FET3.G; no longer FET3.GATE
- net GL: now also FET2.G; no longer FET2.GATE
- net GND: now also IC2.VSS, J2.2, JP1.3; no longer C38.P$2, C39.P$2, IC12.VSS, JP1.2, LS3.GND, SENSOR.4, U$48.2
- net GU: now also FET1.G; no longer FET1.GATE
- net I2C_SCL: now also IC2.P0.27; no longer IC12.P0.27, SENSOR.3, U1.SCL
- net I2C_SDA: now also IC2.P0.26; no longer IC12.P0.26, R7.2, R8.2, SENSOR.2, U1.SDA
- net LED: now also IC2.P0.15; no longer IC12.P0.15
- net MISO: now also IC2.P0.29/AIN5; no longer IC12.P0.29/AIN5
- net MOSI: now also IC2.P0.30/AIN6; no longer IC12.P0.30/AIN6
- net N$1: now also FET3.D; no longer FET3.DRAIN
- net N$3: now also IC3.!SHDN!, SJ1.2; no longer C30.P$1, IC8.VM, R12.1
- net N$50: now also IC2.P0.25; no longer IC12.P0.25
- net N$6: now also FET2.S; no longer FET2.SOURCE
- net NC: now also IC2.NC; no longer IC12.NC
- net OSC_ENABLE: now also JP6.2, SJ1.1; no longer IC3.!SHDN!
- net OUT: now also FET1.S, FET1.SR, FET2.D; no longer FET1.SOURCE, FET1.SOURCE-RETURN, FET2.DRAIN
- net P00: now also IC2.P0.00/XL1; no longer C38.P$1, IC12.P0.00/XL1, Y2.2
- net P01: now also IC2.P0.01/XL2; no longer C39.P$1, IC12.P0.01/XL2, Y2.1
- net P02: now also IC2.P0.02/AIN0; no longer IC12.P0.02/AIN0
- net P03: now also IC2.P0.03/AIN1; no longer IC12.P0.03/AIN1
- net P04: now also IC2.P0.04/AIN2; no longer IC12.P0.04/AIN2
- net P05: now also IC2.P0.05/AIN3; no longer IC12.P0.05/AIN3, UART_INTERFACE.3
- net P06: now also IC2.P0.06, JP1.2; no longer IC12.P0.06, UART_INTERFACE.2
- net P07: now also IC2.P0.07; no longer IC12.P0.07, UART_INTERFACE.4
- net P08: now also IC2.P0.08, JP1.1; no longer IC12.P0.08, UART_INTERFACE.1
- net P09: now also IC2.P0.09/NFC1; no longer IC12.P0.09/NFC1
- net P10: now also IC2.P0.10/NFC2; no longer IC12.P0.10/NFC2
- net P11: now also IC2.P0.11; no longer IC12.P0.11
- net P12: now also IC2.P0.12; no longer IC12.P0.12
- net P13: now also IC2.P0.13; no longer IC12.P0.13
- net P14: now also IC2.P0.14; no longer IC12.P0.14
- net P16: now also IC2.P0.16; no longer IC12.P0.16
- net P17: now also IC2.P0.17; no longer IC12.P0.17
- net P19: now also IC2.P0.19; no longer IC12.P0.19
- net P22: now also IC2.P0.22; no longer IC12.P0.22
- net P23: now also IC2.P0.23; no longer IC12.P0.23
- net P24: now also IC2.P0.24; no longer IC12.P0.24
- net P28: now also IC2.P0.28/AIN4; no longer IC12.P0.28/AIN4
- net SCK: now also IC2.P0.31/AIN7; no longer IC12.P0.31/AIN7
- net SCL: no longer J2.9
- net SDA: no longer J2.10
- net SWDCLK: now also IC2.SWDCLK; no longer IC12.SWDCLK
- net SWDIO: now also IC2.SWDIO; no longer IC12.SWDIO
- net SWO/TDO: now also IC2.P0.18; no longer IC12.P0.18
- net VAMP: now also FET1.D; no longer FET1.DRAIN, J2.1, J2.2, J2.4, R12.2, R16.2
- net VDD_BLE: now also IC2.VDD; no longer IC12.VDD, LS3.VIN
- net XC1: now also IC2.XC1(32MHZ); no longer IC12.XC1(32MHZ)
- net XC2: now also IC2.XC2(32MHZ); no longer IC12.XC2(32MHZ)
Other:
- note added: "# Disable SMPS (external inductors not soldered) CONFIG_BOARD_ENABLE_DCDC=n # Use internal 32k oscillator (no external crystal) CONFIG_CLOCK_CONTROL_NRF_K32SRC_RC=y"
- note added: "ANALOG"
- note added: "DIGITAL"
- note added: "GND"
- note removed: "32.768kHz Crystal (RTC)"
- note removed: "3V3 MCU + OSC"
- note removed: "50V"
- note removed: "5V required Gate voltage GAN FETs EPC8010 rectricted to max. 6V"
- note removed: "Add DC/DC converter as power supply for nRF52 nRF will automatically switch between DC/DC and LDO to ensure minimal power consumption"
- note removed: "Amplification 50V/V"
- note removed: "Application note, filter shunt resistor (current measurements). https://www.st.com/resource/en/application_note/an4304-how-to-filter-the-input-of-a-highside-current-sensing-stmicroelectronics.pdf"
- note removed: "BETAFLIGHT current"
- note removed: "CONNECT WITH NRF"
- note removed: "CTS"
- note removed: "FSR = ±2.048 V"
- note removed: "I2C ADC"
- note removed: "IO EXPANDER REQUIRED? PCA9570GMH"
- note removed: "Input voltage will vary during flight"
- note removed: "MOUSER: 609-L-07C15NKV6T"
- note removed: "MOUSER: 81-LQM18FN100M00D"
- note removed: "NRF52832 CTS"
- note removed: "NRF52832 RTS"
- note removed: "RTS"
- note removed: "Resistor values should be equal!"
- note removed: "SEPIC current"
- note removed: "Sense Amplifier"
- note removed: "approx. 10 - 16.8 V"
- note removed: "buck (boost) converter"
- note removed: "digi pot"
- note removed: "https://www.infineon.com/dgdl/Infineon-AN91445_Antenna_Design_and_RF_Layout_Guidelines-ApplicationNotes-v09_00-EN.pdf"
- moved on the sheet: C8, C9, D4, LS3, R3, SJ1

Commit message: Update PTU firmware and hardware
Parts:
- removed C42, C48, C49, C50: 100n, microbuilder:CAP_CERAMIC0402
- removed C46, C47: 12p, microbuilder:CAP_CERAMIC0402
- removed JP10, JP11, JP12, JP13, JP14, JP6, JP7, JP8, JP9: JUMPER-SMT_2_NO_NO-SILK, SparkFun-Jumpers:JUMPER-SMT_2_NO_NO-SILK
- removed JP4: (no value), microbuilder:SOLDERJUMPERREFLOW_NOPASTE
- removed LS3: MIC94081YFT-TR, MIC94081YFT-TR:MIC94081YFT-TR
- removed R15: 10k, microbuilder:RESISTOR0402
- removed R25: 100k, microbuilder:RESISTOR0603
- removed R26: 10k, microbuilder:RESISTOR0603
- removed UPDATE: (no value), Eagle_SWITCHES (rev18c):434111043826
- added C3, C4: 100n, microbuilder:CAP_CERAMIC0402
- added L2: 742792692, PowerMagnetics (rev18e):WE-CBF_0603_742792692_WB_HS
- added POWER: JUMPER-SMT_2_NO_NO-SILK, SparkFun-Jumpers:JUMPER-SMT_2_NO_NO-SILK
- added R10: 100k, microbuilder:RESISTOR0402
- added R7, R8, R9: 10k, microbuilder:RESISTOR0402
- added TP10, TP11, TP12, TP4, TP6, TP7, TP9: TPTP10SQ, testpad:TPTP10SQ
- added TP3, TP8: TPTP20SQ, testpad:TPTP20SQ
- C21, C22, C5, C8, C9: device microbuilder:CAP_CERAMIC0603 -> microbuilder:CAP_CERAMIC0402
- R3: device microbuilder:RESISTOR0603 -> microbuilder:RESISTOR0402
- TP5: value TPTP20SQ -> TPTP10SQ; device testpad:TPTP20SQ -> testpad:TPTP10SQ
Connections:
- removed net N$10: JP8.2
- removed net N$11: JP9.2
- removed net N$12: JP10.2
- removed net N$13: JP11.2
- removed net N$15: JP13.2
- removed net N$16: JP14.2
- removed net N$50: C47.P$1, IC2.P0.25
- removed net N$6: FET2.S
- removed net N$9: JP7.2
- removed net OSC: IC5.B, IC6.B
- removed net P02: C48.P$1, IC2.P0.02/AIN0, JP12.1
- removed net P03: C49.P$1, IC2.P0.03/AIN1, JP13.1
- removed net P04: C50.P$1, IC2.P0.04/AIN2, JP14.1
- removed net P11: IC2.P0.11, JP6.1
- new net N$14: L2.1, POWER.2
- new net P25: IC2.P0.25
- new net V-5V: C3.P$1, IC2.P0.04/AIN2, R7.2, R8.1
- net +3V3: now also POWER.1, TP6.TP; no longer JP4.1
- net +5V: now also R8.2, TP4.TP
- net AGND: now also FET2.S, R9.1, TP7.TP, TP8.TP; no longer R26.1
- net GND: now also C3.P$2, C4.P$2, R7.1; no longer C42.P$2, C46.P$2, C47.P$2, C48.P$2, C49.P$2, C50.P$2, UPDATE.1
- net I2C_SDA: no longer C46.P$1
- net OSC_CLK: now also IC5.B, IC6.B
- net OSC_ENABLE: now also IC2.P0.11; no longer JP6.2
- net P12: now also TP9.TP; no longer JP7.1
- net P13: now also TP10.TP; no longer JP8.1
- net P14: now also TP11.TP; no longer JP9.1
- net P16: no longer C42.P$1, R15.1, UPDATE.2
- net P17: now also TP12.TP; no longer JP10.1
- net P19: no longer JP11.1
- net V-VAMP: now also C4.P$1, IC2.P0.02/AIN0, R10.1, R9.2; no longer JP12.2, R25.1, R26.2
- net VAMP: now also R10.2, TP3.TP; no longer R25.2
- net VDD_BLE: now also IC2.P0.03/AIN1, L2.2; no longer JP4.2, R15.2
Other:
- note added: "TEST I2C WORKS PERFECT WITHOUT 12pF caps?"
