File: hardware/power-transmitting-unit/PTU-board/design1.sch (EAGLE design)
At the start: 86 parts, among them IC1 LM5113SDX/NOPB, IC2 NRF52832, IC3 DSC1001DI2-006.7800, IC5 74LVC1G00GW, IC6 74LVC1G08GW, J1 62201021121, J2 636101111001, Y1 32MHz

Commit message: Update HW PTU
Parts:
- removed C42, C48, C50: 100n, microbuilder:CAP_CERAMIC0402
- removed JP1: (no value), microbuilder:HEADER-1X3ROUND
- removed JP10, JP11, JP2, JP7, JP8, JP9: JUMPER-SMT_2_NO_NO-SILK, SparkFun-Jumpers:JUMPER-SMT_2_NO_NO-SILK
- removed LS3: MIC94081YFT-TR, MIC94081YFT-TR:MIC94081YFT-TR
- removed R15: 10k, microbuilder:RESISTOR0402
- removed UPDATE: (no value), Eagle_SWITCHES (rev18c):434111043826
- added C3, C4: 100n, microbuilder:CAP_CERAMIC0402
- added L2: 742792692, PowerMagnetics (rev18e):WE-CBF_0603_742792692_WB_HS
- added P14, P15, P16, P17: TPTP10SQ, testpad:TPTP10SQ
- added POWER: JUMPER-SMT_2_NO_NO-SILK, SparkFun-Jumpers:JUMPER-SMT_2_NO_NO-SILK
- added SJ2: SOLDERJUMPERNO, SparkFun-Retired:SOLDERJUMPERNO
- added UART: (no value), microbuilder:HEADER-1X3ROUND
- C21, C22, C5, C8, C9: device microbuilder:CAP_CERAMIC0603 -> microbuilder:CAP_CERAMIC0402
- R3: device microbuilder:RESISTOR0603 -> microbuilder:RESISTOR0402
- TP4, TP5, TP6, TP7: value TPTP20SQ -> TPTP10SQ; device testpad:TPTP20SQ -> testpad:TPTP10SQ
Connections:
- net EN_SENS renamed P20
- removed net MISO: IC2.P0.29/AIN5
- removed net MOSI: IC2.P0.30/AIN6
- removed net N$10: JP8.2
- removed net N$11: JP9.2
- removed net N$12: JP10.2
- removed net N$13: JP11.2
- removed net N$20: LED1.A, R14.1
- removed net N$6: FET2.S
- removed net N$9: JP7.2
- removed net OSC: IC5.B, IC6.B
- removed net P13: IC2.P0.13, JP8.1
- removed net P28: IC2.P0.28/AIN4
- removed net SCL: J1.9
- removed net SDA: J1.10
- new net N$14: L2.1, POWER.2
- new net N$5: LED1.C, R14.2
- new net OUT_GU: C9.P$2, D4.A, FET1.SR, IC1.HS
- new net P03: IC2.P0.03/AIN1
- new net P04: IC2.P0.04/AIN2
- new net P11: IC2.P0.11
- new net P15: IC2.P0.15, P15.TP
- net +3V3: now also POWER.1; no longer JP2.1
- net AGND: now also FET2.S, SJ2.2; no longer C1.P$2, C18.P$2, C2.P$2, C21.P$2, C22.P$2, C5.P$2, C7.P$2, C8.P$2, FET2.SR, IC1.EP, IC1.VSS, IC3.GND, IC5.GND, IC6.GND, J1.3, J1.7, J1.8, R9.1, TP7.TP
- net GND: now also C1.P$2, C18.P$2, C2.P$2, C21.P$2, C22.P$2, C3.P$2, C4.P$2, C5.P$2, C7.P$2, C8.P$2, FET2.SR, IC1.EP, IC1.VSS, IC3.GND, IC5.GND, IC6.GND, J1.3, J1.7, J1.8, R14.1, R9.1, SJ2.1, TP7.TP, UART.3; no longer C42.P$2, C48.P$2, C50.P$2, JP1.3, LED1.C, UPDATE.1
- net I2C_SCL: now also J1.9
- net I2C_SDA: now also J1.10
- net LED: now also IC2.P0.13, LED1.A; no longer IC2.P0.15, R14.2
- net OSC_CLK: now also IC5.B, IC6.B
- net OSC_ENABLE: now also IC2.P0.28/AIN4; no longer IC2.P0.11
- net OUT: no longer C9.P$2, D4.A, FET1.SR, IC1.HS
- net P06: now also UART.1; no longer JP1.2
- net P08: now also UART.2; no longer JP1.1
- net P12: no longer JP7.1
- net P14: now also P14.TP; no longer JP9.1
- net P16: now also P16.TP; no longer C42.P$1, R15.1, UPDATE.2
- net P17: now also P17.TP; no longer JP10.1
- net P19: no longer JP11.1
- net V-5V: now also C3.P$1, IC2.P0.30/AIN6; no longer C50.P$1, IC2.P0.04/AIN2
- net V-VAMP: now also C4.P$1, IC2.P0.29/AIN5; no longer C48.P$1, IC2.P0.02/AIN0
- net VDD_BLE: now also IC2.P0.02/AIN0, L2.2; no longer IC2.P0.03/AIN1, JP2.2, R15.2
Other:
- note removed: "Button"
- note removed: "TEST I2C WORKS PERFECT WITHOUT 12pF caps?"
